File: eagle/Crimea-v2.brd (EAGLE design)
At the start: 160 x 100 mm, 33 parts, among them IC1 ICL7660CSA

Commit message: pcm2707 schematic pre finished
Parts:
- added PCM2707-1:C2, PCM2707-1:C5: 10uF, SparkFun-Passives:CPOL-RADIAL-100UF-25V
- added PCM2707-1:C3, PCM2707-1:C4: 0.1uF, SparkFun-Passives:1206
- added PCM2707-1:C6, PCM2707-1:C7: 1uF, SparkFun-Passives:1206
- added PCM2707-1:R5, PCM2707-1:R7, PCM2707-1:R8: 1.5K, SparkFun-Passives:0805
- added PCM2707-1:R6: 1M, SparkFun-Passives:0805
- added PCM2707-1:Y1: 12MHz CSTCE12MOG52-R0, SparkFun-Clocks:RESONATOR-SMD-3.2X1.3
- PCM2707-1:C1: value 0.1uF -> 10uF; device SparkFun-Passives:EIA3216-KIT -> SparkFun-Passives:CPOL-RADIAL-100UF-25V
- moved PCM2707-1:C1 36.4 mm to (-28.8, -85.0)
Connections:
- new net PCM2707-1:!SUSPEND!: PCM2707-1:U$1.11
- new net PCM2707-1:BCK: PCM2707-1:U$1.19
- new net PCM2707-1:DIN: PCM2707-1:U$1.4
- new net PCM2707-1:DOUT: PCM2707-1:U$1.17
- new net PCM2707-1:LRCK: PCM2707-1:U$1.5
- new net PCM2707-1:N$1: PCM2707-1:R6.1, PCM2707-1:U$1.12, PCM2707-1:Y1.1
- new net PCM2707-1:N$2: PCM2707-1:R5.1, PCM2707-1:U$2.3
- new net PCM2707-1:N$3: PCM2707-1:R6.2, PCM2707-1:U$1.13, PCM2707-1:Y1.3
- new net PCM2707-1:N$6: PCM2707-1:C5.1, PCM2707-1:U$1.32
- new net PCM2707-1:N$7: PCM2707-1:R7.2, PCM2707-1:U$1.15
- new net PCM2707-1:N$8: PCM2707-1:R8.1, PCM2707-1:U$1.10
- new net PCM2707-1:SPI_!SS!: PCM2707-1:U$1.6
- new net PCM2707-1:SPI_CLCK: PCM2707-1:U$1.7
- new net PCM2707-1:SPI_MOSI: PCM2707-1:U$1.8
- new net PCM2707-1:SYSCK: PCM2707-1:U$1.18
- new net PCM2707-1:VOUT_L: PCM2707-1:U$1.28
- new net PCM2707-1:VOUT_R: PCM2707-1:U$1.29
- net PCM2707-1:3.3V: now also PCM2707-1:C1.1, PCM2707-1:C2.1, PCM2707-1:C3.1, PCM2707-1:C4.1, PCM2707-1:C6.2, PCM2707-1:C7.1, PCM2707-1:R7.1, PCM2707-1:R8.2, PCM2707-1:U$1.2, PCM2707-1:U$1.27, PCM2707-1:U$1.30; no longer PCM2707-1:C1.A, PCM2707-1:R4.1, PCM2707-1:U$2.2
- net PCM2707-1:DGND: now also PCM2707-1:C7.2, PCM2707-1:U$1.25, PCM2707-1:U$1.26
- net PCM2707-1:GNDA: now also PCM2707-1:C1.2, PCM2707-1:C2.2, PCM2707-1:C3.2, PCM2707-1:C4.2, PCM2707-1:C5.2, PCM2707-1:C6.1, PCM2707-1:U$1.1, PCM2707-1:U$1.31, PCM2707-1:U$1.9, PCM2707-1:Y1.2; no longer PCM2707-1:C1.C
- net PCM2707-1:USB_D+: now also PCM2707-1:R5.2; no longer PCM2707-1:U$2.3
- net PCM2707-1:USB_VBUS: now also PCM2707-1:R4.1, PCM2707-1:U$1.3, PCM2707-1:U$2.2

Commit message: pcm2707 DGND error fixed
Connections:
- removed net PCM2707-1:GNDA: PCM2707-1:C1.2, PCM2707-1:C2.2, PCM2707-1:C3.2, PCM2707-1:C4.2, PCM2707-1:C5.2, PCM2707-1:C6.1, PCM2707-1:U$1.1, PCM2707-1:U$1.20, PCM2707-1:U$1.31, PCM2707-1:U$1.9, PCM2707-1:Y1.2
- net PCM2707-1:DGND: now also PCM2707-1:C1.2, PCM2707-1:C2.2, PCM2707-1:C3.2, PCM2707-1:C4.2, PCM2707-1:C5.2, PCM2707-1:C6.1, PCM2707-1:U$1.1, PCM2707-1:U$1.20, PCM2707-1:U$1.31, PCM2707-1:U$1.9, PCM2707-1:Y1.2
Changed lines of the file:
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@@
 <contactref element="PCM2707-1:C7" pad="2"/>
 <contactref element="PCM2707-1:U$1" pad="26"/>
-<wire x1="-3.186" y1="-53.34" x2="-54.734" y2="-106.68" width="0" layer="19" extent="1-1"/>
-<wire x1="16.256" y1="-45.974" x2="-3.186" y2="-53.34" width="0" layer="19" extent="1-1"/>
-<wire x1="8.515" y1="-34.3916" x2="16.256" y2="-45.974" width="0" layer="19" extent="1-1"/>
-<wire x1="8.515" y1="-25.8064" x2="8.515" y2="-34.3916" width="0" layer="19" extent="1-1"/>
+<contactref element="PCM2707-1:U$1" pad="20"/>
+<contactref element="PCM2707-1:U$1" pad="9"/>
+<contactref element="PCM2707-1:Y1" pad="2"/>
+<contactref element="PCM2707-1:U$1" pad="1"/>
+<contactref element="PCM2707-1:C1" pad="2"/>
+<contactref element="PCM2707-1:C4" pad="2"/>
+<contactref element="PCM2707-1:C2" pad="2"/>
+<contactref element="PCM2707-1:C3" pad="2"/>
+<contactref element="PCM2707-1:C5" pad="2"/>
+<contactref element="PCM2707-1:C6" pad="1"/>
+<contactref element="PCM2707-1:U$1" pad="31"/>
+<wire x1="-52.454" y1="-106.68" x2="-54.734" y2="-106.68" width="0" layer="19" extent="1-1"/>
+<wire x1="-40.132" y1="-101.473" x2="-52.454" y2="-106.68" width="0" layer="19" extent="1-1"/>
+<wire x1="-39.494" y1="-90.17" x2="-40.132" y2="-101.473" width="0" layer="19" extent="1-1"/>
+<wire x1="-44.574" y1="-90.17" x2="-39.494" y2="-90.17" width="0" layer="19" extent="1-1"/>
+<wire x1="-30.099" y1="-84.963" x2="-39.494" y2="-90.17" width="0" layer="19" extent="1-1"/>
+<wire x1="-30.099" y1="-68.453" x2="-30.099" y2="-84.963" width="0" layer="19" extent="1-1"/>
+<wire x1="-23.114" y1="-57.023" x2="-30.099" y2="-68.453" width="0" layer="19" extent="1-1"/>
+<wire x1="-3.186" y1="-53.34" x2="-23.114" y2="-57.023" width="0" layer="19" extent="1-1"/>
+<wire x1="2.915" y1="-34.3916" x2="-3.186" y2="-53.34" width="0" layer="19" extent="1-1"/>
+<wire x1="8.515" y1="-34.3916" x2="2.915" y2="-34.3916" width="0" layer="19" extent="1-1"/>
+<wire x1="10.0076" y1="-30.499" x2="8.515" y2="-34.3916" width="0" layer="19" extent="1-1"/>
+<wire x1="8.515" y1="-25.8064" x2="10.0076" y2="-30.499" width="0" layer="19" extent="1-1"/>
 <wire x1="7.715" y1="-25.8064" x2="8.515" y2="-25.8064" width="0" layer="19" extent="1-1"/>
+<wire x1="3.715" y1="-25.8064" x2="7.715" y2="-25.8064" width="0" layer="19" extent="1-1"/>
+<wire x1="1.4224" y1="-27.299" x2="3.715" y2="-25.8064" width="0" layer="19" extent="1-1"/>
+<wire x1="16.256" y1="-45.974" x2="8.515" y2="-34.3916" width="0" layer="19" extent="1-1"/>
 </signal>
 <signal name="PCM2707-1:USB_VBUS">
@@
 <wire x1="10.0076" y1="-29.699" x2="6.915" y2="-25.8064" width="0" layer="19" extent="1-1"/>
 </signal>
-<signal name="PCM2707-1:GNDA">
-<contactref element="PCM2707-1:U$1" pad="20"/>
-<contactref element="PCM2707-1:U$1" pad="9"/>
-<contactref element="PCM2707-1:Y1" pad="2"/>
-<contactref element="PCM2707-1:U$1" pad="1"/>
-<contactref element="PCM2707-1:C1" pad="2"/>
-<contactref element="PCM2707-1:C4" pad="2"/>
-<contactref element="PCM2707-1:C2" pad="2"/>
-<contactref element="PCM2707-1:C3" pad="2"/>
-<contactref element="PCM2707-1:C5" pad="2"/>
-<contactref element="PCM2707-1:C6" pad="1"/>
-<contactref element="PCM2707-1:U$1" pad="31"/>
-<wire x1="-40.132" y1="-101.473" x2="-52.454" y2="-106.68" width="0" layer="19" extent="1-1"/>
-<wire x1="-39.494" y1="-90.17" x2="-40.132" y2="-101.473" width="0" layer="19" extent="1-1"/>
-<wire x1="-44.574" y1="-90.17" x2="-39.494" y2="-90.17" width="0" layer="19" extent="1-1"/>
-<wire x1="-30.099" y1="-84.963" x2="-39.494" y2="-90.17" width="0" layer="19" extent="1-1"/>
-<wire x1="-30.099" y1="-68.453" x2="-30.099" y2="-84.963" width="0" layer="19" extent="1-1"/>
-<wire x1="-23.114" y1="-57.023" x2="-30.099" y2="-68.453" width="0" layer="19" extent="1-1"/>
-<wire x1="2.915" y1="-34.3916" x2="-23.114" y2="-57.023" width="0" layer="19" extent="1-1"/>
-<wire x1="1.4224" y1="-27.299" x2="2.915" y2="-34.3916" width="0" layer="19" extent="1-1"/>
-<wire x1="3.715" y1="-25.8064" x2="1.4224" y2="-27.299" width="0" layer="19" extent="1-1"/>
-<wire x1="10.0076" y1="-30.499" x2="3.715" y2="-25.8064" width="0" layer="19" extent="1-1"/>
-</signal>
 <signal name="PCM2707-1:PULLUP_HANDLE">
