File: eagle/Crimea-v2.brd (EAGLE design)
At the start: 160 x 100 mm, 44 parts, among them IC1 ICL7660CSA

Commit message: minor changes
Parts:
- added PCM2707-1:R9: 1M, SparkFun-Passives:0805
- moved PCM2707-1:C1 135.5 mm to (-58.3, 47.2)
- moved PCM2707-1:C3 135.5 mm to (-70.4, 42.0)
- moved PCM2707-1:C4 135.5 mm to (-75.4, 42.0)
- moved PCM2707-1:C6 135.5 mm to (-80.5, 25.5)
- moved PCM2707-1:C7 135.5 mm to (-85.6, 25.5)
- moved PCM2707-1:C5 135.5 mm to (-68.3, 30.7)
- moved PCM2707-1:C2 87.4 mm to (-75.4, 5.46)
- moved PCM2707-1:R1 87.4 mm to (-48.9, 20.6)
- moved PCM2707-1:R3 87.4 mm to (-55.0, 20.6)
- moved PCM2707-1:R5 87.4 mm to (-66.2, 15.7)
- moved PCM2707-1:R6 87.4 mm to (-77.3, 15.7)
- moved PCM2707-1:R7 87.4 mm to (-80.4, 15.7)
- moved PCM2707-1:U$2 87.4 mm to (-59.1, 17.8)
- moved PCM2707-1:J1 87.4 mm to (-38.0, 27.9)
- moved PCM2707-1:R2 87.4 mm to (-51.9, 20.6)
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Connections:
- new net PCM2707-1:N$9: PCM2707-1:R9.2, PCM2707-1:U$1.3
- net PCM2707-1:USB_VBUS: now also PCM2707-1:R9.1; no longer PCM2707-1:U$1.3

Commit message: inverter deleted. dac added. it is not finished yet
Parts:
- removed C1, C2: (no value), SparkFun-Passives:EIA3216-KIT
- removed C_OSC: (no value), SparkFun-Passives:1206
- removed I2S_CONVERTER:U$3: PCM1794A, EduAreaLib:SSOP28-0.65-10.2X5.2MM
- removed IC1: ICL7660CSA, maxim:SO08
- added DAC1:C1, DAC1:C2, DAC1:C6: 10uF, SparkFun-Passives:CPOL-RADIAL-100UF-25V
- added DAC1:C3, DAC1:C4, DAC1:C5: 0.1uF, SparkFun-Passives:1206
- added DAC1:U$1: PCM1794A, EduAreaLib:SSOP28-0.65-10.2X5.2MM
Connections:
- removed net +5V: C_OSC.2, IC1.8
- removed net -5V: C2.C, IC1.5
- removed net GND: C2.A, IC1.3
- removed net I2S_CONVERTER:BCK: I2S_CONVERTER:U$3.6
- removed net I2S_CONVERTER:DATA: I2S_CONVERTER:U$3.5
- removed net I2S_CONVERTER:LRCK: I2S_CONVERTER:U$3.4
- removed net I2S_CONVERTER:SCK: I2S_CONVERTER:U$3.7
- removed net N$10: C1.A, IC1.2
- removed net N$2: C_OSC.1, IC1.7
- removed net N$3: C1.C, IC1.4
- new net DAC1:!RST!: DAC1:U$1.14
- new net DAC1:3.3V: DAC1:C2.1, DAC1:C4.2, DAC1:U$1.9
- new net DAC1:5V: DAC1:C1.1, DAC1:C3.1, DAC1:C5.2, DAC1:C6.1, DAC1:U$1.15, DAC1:U$1.28
- new net DAC1:AGND: DAC1:C1.2, DAC1:C3.2, DAC1:C5.1, DAC1:C6.2, DAC1:U$1.16, DAC1:U$1.27
- new net DAC1:BCK: DAC1:U$1.6
- new net DAC1:CHSL: DAC1:U$1.2
- new net DAC1:DATA: DAC1:U$1.5
- new net DAC1:DEM: DAC1:U$1.3
- new net DAC1:DGND: DAC1:C2.2, DAC1:C4.1, DAC1:U$1.8
- new net DAC1:FMT0: DAC1:U$1.11
- new net DAC1:FMT1: DAC1:U$1.12
- new net DAC1:LRCK: DAC1:U$1.4
- new net DAC1:MONO: DAC1:U$1.1
- new net DAC1:MUTE: DAC1:U$1.10
- new net DAC1:SYSCK: DAC1:U$1.7
- new net DAC1:ZERO: DAC1:U$1.13
Routing:
- net GND: track 6.13 -> 0.00 mm
- net -5V: track 4.43 -> 0.00 mm
- net N$2: track 3.47 -> 0.00 mm
- net +5V: track 3.47 -> 0.00 mm
- net N$3: track 3.36 -> 0.00 mm
- net N$10: track 3.25 -> 0.00 mm
Changed lines of the file:
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@@
 <drawing>
 <settings>
-<setting alwaysvectorfont="yes"/>
+<setting alwaysvectorfont="no"/>
 <setting keepoldvectorfont="yes"/>
 <setting verticaltext="up"/>
@@
 </autorouter>
 <elements>
-<element name="IC1" library="maxim" library_urn="urn:adsk.eagle:library:269" package="SO08" value="ICL7660CSA" x="75.819" y="9.017">
-<attribute name="MF" value="MAXIM" x="75.819" y="9.017" size="1.778" layer="27" display="off"/>
-<attribute name="MPN" value="ICL7660CSA" x="75.819" y="9.017" size="1.778" layer="27" display="off"/>
-<attribute name="OC_FARNELL" value="9724710" x="75.819" y="9.017" size="1.778" layer="27" display="off"/>
-<attribute name="OC_NEWARK" value="34C3732" x="75.819" y="9.017" size="1.778" layer="27" display="off"/>
-</element>
-<element name="C_OSC" library="SparkFun-Passives" package="1206" value="" x="74.549" y="15.24" rot="R180"/>
-<element name="C1" library="SparkFun-Passives" package="EIA3216-KIT" value="" x="76.581" y="2.794" rot="R180"/>
-<element name="C2" library="SparkFun-Passives" package="EIA3216-KIT" value="" x="80.772" y="9.017" rot="R270"/>
-<element name="I2S_CONVERTER:U$3" library="EduAreaLib" package="SSOP28-0.65-10.2X5.2MM" value="PCM1794A" x="102.87" y="-18.034"/>
 <element name="VR:J1" library="SparkFun-Connectors" package="1X03_LONGPADS" value="" x="13.716" y="21.844" rot="R180"/>
 <element name="VR:B1" library="rectifier" library_urn="urn:adsk.eagle:library:336" package="SOIC-4" value="MB6S" x="10.922" y="28.321" rot="R270"/>
@@
 <element name="PCM2707-1:C7" library="SparkFun-Passives" package="1206" value="1uF" x="-85.598" y="25.527"/>
 <element name="PCM2707-1:R9" library="SparkFun-Passives" package="0805" value="1M" x="-89.535" y="-21.59"/>
+<element name="DAC1:U$1" library="EduAreaLib" package="SSOP28-0.65-10.2X5.2MM" value="PCM1794A" x="-83.947" y="-29.337"/>
+<element name="DAC1:C2" library="SparkFun-Passives" package="CPOL-RADIAL-100UF-25V" value="10uF" x="-81.534" y="-43.307"/>
+<element name="DAC1:C4" library="SparkFun-Passives" package="1206" value="0.1uF" x="-88.519" y="-54.61"/>
+<element name="DAC1:C1" library="SparkFun-Passives" package="CPOL-RADIAL-100UF-25V" value="10uF" x="-81.534" y="-65.913"/>
+<element name="DAC1:C3" library="SparkFun-Passives" package="1206" value="0.1uF" x="-93.599" y="-71.12"/>
+<element name="DAC1:C5" library="SparkFun-Passives" package="1206" value="0.1uF" x="-98.679" y="-71.12"/>
+<element name="DAC1:C6" library="SparkFun-Passives" package="CPOL-RADIAL-100UF-25V" value="10uF" x="-91.567" y="-82.423"/>
 </elements>
 <signals>
-<signal name="GND">
-<contactref element="IC1" pad="3"/>
-<contactref element="C2" pad="A"/>
-<wire x1="76.454" y1="5.9436" x2="76.454" y2="7.493" width="0.6096" layer="1"/>
-<wire x1="76.454" y1="7.493" x2="76.708" y2="7.747" width="0.6096" layer="1"/>
-<wire x1="76.708" y1="7.747" x2="80.392" y2="7.747" width="0.6096" layer="1"/>
-<wire x1="80.392" y1="7.747" x2="80.772" y2="7.367" width="0.6096" layer="1"/>
-</signal>
-<signal name="+5V">
-<contactref element="IC1" pad="8"/>
-<contactref element="C_OSC" pad="2"/>
-<wire x1="73.914" y1="12.0904" x2="73.914" y2="13.208" width="0.6096" layer="1"/>
-<wire x1="73.914" y1="13.208" x2="73.152" y2="13.97" width="0.6096" layer="1"/>
-<wire x1="73.152" y1="13.97" x2="73.152" y2="15.237" width="0.6096" layer="1"/>
-<wire x1="73.152" y1="15.237" x2="73.149" y2="15.24" width="0.6096" layer="1"/>
-</signal>
-<signal name="N$2">
-<contactref element="IC1" pad="7"/>
-<contactref element="C_OSC" pad="1"/>
-<wire x1="75.184" y1="12.0904" x2="75.184" y2="13.335" width="0.6096" layer="1"/>
-<wire x1="75.184" y1="13.335" x2="75.946" y2="14.097" width="0.6096" layer="1"/>
-<wire x1="75.946" y1="14.097" x2="75.946" y2="15.237" width="0.6096" layer="1"/>
-<wire x1="75.946" y1="15.237" x2="75.949" y2="15.24" width="0.6096" layer="1"/>
-</signal>
-<signal name="-5V">
-<contactref element="IC1" pad="5"/>
-<contactref element="C2" pad="C"/>
-<wire x1="77.724" y1="12.0904" x2="77.724" y2="10.922" width="0.6096" layer="1"/>
-<wire x1="77.724" y1="10.922" x2="78.105" y2="10.541" width="0.6096" layer="1"/>
-<wire x1="78.105" y1="10.541" x2="80.646" y2="10.541" width="0.6096" layer="1"/>
-<wire x1="80.646" y1="10.541" x2="80.772" y2="10.667" width="0.6096" layer="1"/>
-</signal>
-<signal name="N$3">
-<contactref element="IC1" pad="4"/>
-<contactref element="C1" pad="C"/>
-<wire x1="78.231" y1="2.794" x2="78.231" y2="3.684" width="0.6096" layer="1"/>
-<wire x1="78.231" y1="3.684" x2="77.724" y2="4.191" width="0.6096" layer="1"/>
-<wire x1="77.724" y1="4.191" x2="77.724" y2="5.9436" width="0.6096" layer="1"/>
-</signal>
-<signal name="N$10">
-<contactref element="C1" pad="A"/>
-<contactref element="IC1" pad="2"/>
-<wire x1="74.931" y1="2.794" x2="74.931" y2="4.192" width="0.6096" layer="1"/>
-<wire x1="74.931" y1="4.192" x2="75.184" y2="4.445" width="0.6096" layer="1"/>
-<wire x1="75.184" y1="4.445" x2="75.184" y2="5.9436" width="0.6096" layer="1"/>
-</signal>
-<signal name="I2S_CONVERTER:SCK">
-<contactref element="I2S_CONVERTER:U$3" pad="7"/>
-</signal>
-<signal name="I2S_CONVERTER:BCK">
-<contactref element="I2S_CONVERTER:U$3" pad="6"/>
-</signal>
-<signal name="I2S_CONVERTER:DATA">
-<contactref element="I2S_CONVERTER:U$3" pad="5"/>
-</signal>
-<signal name="I2S_CONVERTER:LRCK">
-<contactref element="I2S_CONVERTER:U$3" pad="4"/>
-</signal>
 <signal name="VR:EXTGND">
 <contactref element="VR:B2" pad="~1"/>
@@
 <wire x1="-45.1866" y1="45.015" x2="-88.635" y2="-21.59" width="0" layer="19" extent="1-1"/>
 </signal>
+<signal name="DAC1:MONO">
+<contactref element="DAC1:U$1" pad="1"/>
+</signal>
+<signal name="DAC1:CHSL">
+<contactref element="DAC1:U$1" pad="2"/>
+</signal>
+<signal name="DAC1:DEM">
+<contactref element="DAC1:U$1" pad="3"/>
+</signal>
+<signal name="DAC1:LRCK">
+<contactref element="DAC1:U$1" pad="4"/>
+</signal>
+<signal name="DAC1:DATA">
+<contactref element="DAC1:U$1" pad="5"/>
+</signal>
+<signal name="DAC1:BCK">
+<contactref element="DAC1:U$1" pad="6"/>
+</signal>
+<signal name="DAC1:SYSCK">
+<contactref element="DAC1:U$1" pad="7"/>
+</signal>
+<signal name="DAC1:DGND">
+<contactref element="DAC1:U$1" pad="8"/>
+<contactref element="DAC1:C2" pad="2"/>
+<contactref element="DAC1:C4" pad="1"/>
+<wire x1="-82.804" y1="-43.307" x2="-89.919" y2="-54.61" width="0" layer="19" extent="1-1"/>
+<wire x1="-83.622" y1="-32.962" x2="-82.804" y2="-43.307" width="0" layer="19" extent="1-1"/>
+</signal>
+<signal name="DAC1:3.3V">
+<contactref element="DAC1:C2" pad="1"/>
+<contactref element="DAC1:U$1" pad="9"/>
+<contactref element="DAC1:C4" pad="2"/>
+<wire x1="-80.264" y1="-43.307" x2="-87.119" y2="-54.61" width="0" layer="19" extent="1-1"/>
+<wire x1="-82.972" y1="-32.962" x2="-80.264" y2="-43.307" width="0" layer="19" extent="1-1"/>
+</signal>
+<signal name="DAC1:MUTE">
+<contactref element="DAC1:U$1" pad="10"/>
+</signal>
+<signal name="DAC1:FMT0">
+<contactref element="DAC1:U$1" pad="11"/>
+</signal>
+<signal name="DAC1:FMT1">
+<contactref element="DAC1:U$1" pad="12"/>
+</signal>
+<signal name="DAC1:ZERO">
+<contactref element="DAC1:U$1" pad="13"/>
+</signal>
+<signal name="DAC1:!RST!">
+<contactref element="DAC1:U$1" pad="14"/>
+</signal>
+<signal name="DAC1:5V">
+<contactref element="DAC1:U$1" pad="28"/>
+<contactref element="DAC1:C3" pad="1"/>
+<contactref element="DAC1:C1" pad="1"/>
+<contactref element="DAC1:C5" pad="2"/>
+<contactref element="DAC1:C6" pad="1"/>
+<contactref element="DAC1:U$1" pad="15"/>
+<wire x1="-94.999" y1="-71.12" x2="-90.297" y2="-82.423" width="0" layer="19" extent="1-1"/>
+<wire x1="-97.279" y1="-71.12" x2="-94.999" y2="-71.12" width="0" layer="19" extent="1-1"/>
+<wire x1="-80.264" y1="-65.913" x2="-94.999" y2="-71.12" width="0" layer="19" extent="1-1"/>
+<wire x1="-79.722" y1="-25.712" x2="-80.264" y2="-65.913" width="0" layer="19" extent="1-1"/>
+<wire x1="-88.172" y1="-25.712" x2="-79.722" y2="-25.712" width="0" layer="19" extent="1-1"/>
+</signal>
+<signal name="DAC1:AGND">
+<contactref element="DAC1:U$1" pad="27"/>
+<contactref element="DAC1:C1" pad="2"/>
+<contactref element="DAC1:C3" pad="2"/>
+<contactref element="DAC1:C6" pad="2"/>
+<contactref element="DAC1:C5" pad="1"/>
+<contactref element="DAC1:U$1" pad="16"/>
+<wire x1="-92.199" y1="-71.12" x2="-92.837" y2="-82.423" width="0" layer="19" extent="1-1"/>
+<wire x1="-100.079" y1="-71.12" x2="-92.199" y2="-71.12" width="0" layer="19" extent="1-1"/>
+<wire x1="-82.804" y1="-65.913" x2="-92.199" y2="-71.12" width="0" layer="19" extent="1-1"/>
+<wire x1="-80.372" y1="-25.712" x2="-82.804" y2="-65.913" width="0" layer="19" extent="1-1"/>
+<wire x1="-87.522" y1="-25.712" x2="-80.372" y2="-25.712" width="0" layer="19" extent="1-1"/>
+</signal>
 </signals>

Commit message: DAC
Parts:
- added DAC1:C10, DAC1:C12, DAC1:C19, DAC1:C20, DAC1:C9: 10uF, SparkFun-Passives:CPOL-RADIAL-100UF-25V
- added DAC1:C11, DAC1:C13, DAC1:C22, DAC1:C23: 0.1uF, SparkFun-Passives:1206
- added DAC1:C14, DAC1:C15, DAC1:C16, DAC1:C17: 2.7nF, SparkFun-Passives:1206
- added DAC1:C18, DAC1:C21: 100uF, SparkFun-Passives:CPOL-RADIAL-100UF-25V
- added DAC1:C7, DAC1:C8: 47uF, SparkFun-Passives:CPOL-RADIAL-100UF-25V
- added DAC1:IC1: OPA4134UA, linear:SO14
- added DAC1:R1: 10K, SparkFun-Passives:0805
- added DAC1:R10, DAC1:R11, DAC1:R12, DAC1:R2, DAC1:R3, DAC1:R4, DAC1:R5, DAC1:R6, DAC1:R7, DAC1:R8: 1K, SparkFun-Passives:0805
- added DAC1:R13, DAC1:R9: 39.2, SparkFun-Passives:0805
- added DAC1:U$6: TPA6120A2, EduAreaLib:SOIC20S
Connections:
- new net DAC1:+12V: DAC1:C10.1, DAC1:C11.2, DAC1:C18.1, DAC1:C19.1, DAC1:C22.1, DAC1:IC1.4, DAC1:U$6.18, DAC1:U$6.3
- new net DAC1:-12V: DAC1:C12.2, DAC1:C13.2, DAC1:C20.2, DAC1:C21.2, DAC1:C23.1, DAC1:IC1.11, DAC1:U$6.1, DAC1:U$6.20
- new net DAC1:LOUT: DAC1:R9.2
- new net DAC1:N$1: DAC1:C14.2, DAC1:IC1.2, DAC1:R2.1, DAC1:U$1.26
- new net DAC1:N$10: DAC1:R10.2, DAC1:R11.2, DAC1:U$6.17
- new net DAC1:N$11: DAC1:R12.2, DAC1:R13.1, DAC1:U$6.19
- new net DAC1:N$14: DAC1:C15.1, DAC1:IC1.7, DAC1:R3.2, DAC1:R6.1
- new net DAC1:N$17: DAC1:C16.2, DAC1:IC1.9, DAC1:R4.1, DAC1:U$1.18
- new net DAC1:N$2: DAC1:C15.2, DAC1:IC1.6, DAC1:R3.1, DAC1:U$1.25
- new net DAC1:N$20: DAC1:C16.1, DAC1:IC1.8, DAC1:R12.1, DAC1:R4.2, DAC1:U$6.16
- new net DAC1:N$23: DAC1:C17.2, DAC1:IC1.13, DAC1:R5.1, DAC1:U$1.17
- new net DAC1:N$25: DAC1:C17.1, DAC1:IC1.14, DAC1:R11.1, DAC1:R5.2
- new net DAC1:N$3: DAC1:R1.1, DAC1:U$1.20
- new net DAC1:N$4: DAC1:R6.2, DAC1:R7.2, DAC1:U$6.4
- new net DAC1:N$5: DAC1:C7.2, DAC1:U$1.22
- new net DAC1:N$6: DAC1:C8.2, DAC1:U$1.21
- new net DAC1:N$8: DAC1:C14.1, DAC1:IC1.1, DAC1:R2.2, DAC1:R8.1, DAC1:U$6.5
- new net DAC1:N$9: DAC1:R8.2, DAC1:R9.1, DAC1:U$6.2
- new net DAC1:ROUT: DAC1:R13.2
- net DAC1:3.3V: now also DAC1:C10.2, DAC1:C11.1, DAC1:C12.1, DAC1:C13.1, DAC1:IC1.10, DAC1:IC1.12, DAC1:IC1.3, DAC1:IC1.5, DAC1:R10.1, DAC1:R7.1
- net DAC1:5V: now also DAC1:C7.1, DAC1:C8.1, DAC1:C9.1, DAC1:U$1.23
- net DAC1:AGND: now also DAC1:C18.2, DAC1:C19.2, DAC1:C20.1, DAC1:C21.1, DAC1:C22.2, DAC1:C23.2, DAC1:C9.2, DAC1:R1.2, DAC1:U$1.19, DAC1:U$1.24

Commit message: added +-5V reg
Parts:
- removed VR:C_IN-: 10uF, SparkFun-Passives:EIA3216-KIT
- added VR:C_IN+1, VR:C_IN-1, VR:C_IN-2, VR:C_OUT+1, VR:C_OUT-1: 10uF, SparkFun-Passives:EIA3216-KIT
- added VR:L3, VR:L4: (no value), SparkFun-Passives:INDUCTOR-1206
- added VR:R10, VR:R7: 10K, SparkFun-Passives:0805
- added VR:R11, VR:R8: 2.7K, SparkFun-Passives:0805
- added VR:R12, VR:R9: ??, SparkFun-Passives:0805
- added VR:U$3: LM2991, EduAreaLib:DDPAK/TO-263
- added VR:U$4: LM2941, EduAreaLib:DDPAK/TO-263
- VR:J2: device SparkFun-Connectors:1X03_LONGPADS -> SparkFun-Connectors:1X05_LONGPADS
- VR:J3: device SparkFun-Connectors:1X01 -> SparkFun-Connectors:MOLEX-1X2
- moved VR:J3 427.0 mm to (-171.2, -357.4)
- moved VR:J2 421.4 mm to (-171.2, -338.6), turned to 0 degrees
Connections:
- removed net VR:!ON!/OFF: VR:J3.1, VR:R1.2, VR:R2.2, VR:U$1.2, VR:U$2.2
- removed net VR:N$6: VR:B2.+, VR:C_IN-.C, VR:U$1.3, VR:U$1.TAB
- new net VR:+-12_!ON!/OFF: VR:J3.2, VR:R1.2, VR:R2.2, VR:U$1.2, VR:U$2.2
- new net VR:+5V: VR:C_OUT+1.A, VR:J2.1, VR:L4.P$2
- new net VR:-5V: VR:C_OUT-1.C, VR:J2.5, VR:L3.P$2
- new net VR:5V_!ON!/OFF: VR:J3.1, VR:R10.2, VR:R7.2, VR:U$3.2, VR:U$4.2
- new net VR:N$1: VR:B2.+, VR:C_IN-1.C, VR:C_IN-2.C, VR:U$1.3, VR:U$1.TAB, VR:U$3.3, VR:U$3.TAB
- new net VR:N$10: VR:R11.1, VR:R12.2, VR:U$4.1
- new net VR:N$11: VR:L4.P$1, VR:R11.2, VR:U$4.5
- new net VR:N$2: VR:R8.1, VR:R9.2, VR:U$3.1
- new net VR:N$3: VR:L3.P$1, VR:R8.2, VR:U$3.5
- net VR:+12V: now also VR:J2.2; no longer VR:J2.1
- net VR:-12V: now also VR:J2.4; no longer VR:J2.3
- net VR:AGND: now also VR:C_IN+1.C, VR:C_IN-1.A, VR:C_IN-2.A, VR:C_OUT+1.C, VR:C_OUT-1.A, VR:J2.3, VR:R10.1, VR:R12.1, VR:R7.1, VR:R9.1, VR:U$3.4, VR:U$4.3, VR:U$4.TAB; no longer VR:C_IN-.A, VR:J2.2
- net VR:N$5: now also VR:C_IN+1.A, VR:U$4.4
Routing:
- net VR:!ON!/OFF: track 32.3 -> 0.00 mm, vias 2 -> 0
- net VR:N$6: track 22.1 -> 0.00 mm
- net VR:+-12_!ON!/OFF: track 0.00 -> 20.9 mm, vias 0 -> 2
- net VR:AGND: track 124.2 -> 112.8 mm
- net VR:+12V: track 27.5 -> 21.3 mm
