File: eagle/Crimea-v2.sch (EAGLE design)
At the start: 4 parts, among them IC1 ICL7660CSA

Commit message: inverter deleted. dac added. it is not finished yet
Parts:
- removed C1, C2: (no value), SparkFun-Passives:CAP_POL1206-KIT
- removed C_OSC: (no value), SparkFun-Passives:CAP1206
- removed IC1: ICL7660CSA, maxim:ICL7660CSA
Connections:
- removed net +5V: C_OSC.2, IC1.V+
- removed net -5V: C2.-, IC1.VOUT
- removed net 3.3V: C1.+, C2.+
- removed net DGND: C1.-, C2.-
- removed net GND: C2.+, IC1.GND
- removed net N$10: C1.+, IC1.CAP+
- removed net N$2: C_OSC.1, IC1.OSC
- removed net N$3: C1.-, IC1.CAP-

Commit message: DAC
Other:
- note added: "I/V Stage"
