File: eagle/power_supply.sch (EAGLE design)
At the start: 34 parts

Commit message: power supply board is finished
Parts:
- renumbered C_IN+ to C_IN+12, C_IN+1 to C_IN+5, C_IN-1 to C_IN-5, C_IN-2 to C_IN-12, C_OUT+ to C_OUT+12, C_OUT+1 to C_OUT+5, C_OUT- to C_OUT-12, C_OUT-1 to C_OUT-5, U$1 to U1, U$2 to U2, U$3 to U3, U$4 to U4

Commit message: power supply finished
Parts:
- C_IN+12, C_IN+5, C_IN-12, C_IN-5: device SparkFun-Passives:CAP_POLPTH1 -> SparkFun-Passives:CAP_POL1206
- R5: value 2.7K -> 23K
- R6, R9: value ?? -> 2.7K
- R8: value 2.7K -> 7.9K
Other:
- note added: "LM2941: Vref=1.275 R11 = R12 * (Vout/Vref - 1) R3 = R4 * (Vout/Vref - 1) LM2991: Vout = Vref× (1+ R2/R1 )-(Iadj*R2)"
- note removed: "LM2941: Vref=1.275 R11 = R12 * (Vout/Vref - 1) R3 = R4 * (Vout/Vref - 1)"
- moved on the sheet: C_IN+5

Commit message: repaint power supply
Parts:
- J1: device SparkFun-Connectors:CONN_03LONGPADS -> SparkFun-Connectors:CONN_04LONGPADS
Connections:
- removed net EXTGND: B1.AC2, B2.AC1, J1.2
- new net N$13: B1.AC2, J1.3
- new net N$6: B2.AC1, J1.2
- net AGND: now also B2.+; no longer B2.-
- net N$1: now also B2.-; no longer B2.+
- net ~15V_PLUS: now also J1.4; no longer J1.3
Other:
- moved on the sheet: B2
