File: eagle/power_supply.brd (EAGLE design)
At the start: 46 x 61 mm, 34 parts, among them U1 LM2991, U2 LM2941, U3 LM2991, U4 LM2941

Commit message: power supply finished
Parts:
- C_IN+12, C_IN+5, C_IN-12, C_IN-5: device SparkFun-Passives:CPOL-RADIAL-100UF-25V -> SparkFun-Passives:EIA3216
- R5: value 2.7K -> 23K
- R6, R9: value ?? -> 2.7K
- R8: value 2.7K -> 7.9K
- moved C_IN-5 9.92 mm to (16.3, 8.35), turned to 0 degrees
- moved C_IN+5 7.65 mm to (20.1, 47.2), turned to 180 degrees
- moved C_IN-12 7.64 mm to (32.2, 7.85), turned to 0 degrees
- moved C_IN+12 6.83 mm to (37.4, 47.4), turned to 180 degrees
- moved R1 3.50 mm to (39.6, 49.6)
- moved R7 3.00 mm to (29.7, 5.66)
- moved R10 2.51 mm to (22.6, 49.4)
- moved R11 2.00 mm to (16.1, 47.1)
- moved R12 2.00 mm to (16.1, 50.2)
- moved R2 2.00 mm to (14.0, 5.96)
- moved R3 2.00 mm to (33.4, 47.2)
- moved R4 2.00 mm to (33.4, 50.2)
- moved R5 2.00 mm to (20.1, 8.51)
- moved R6 2.00 mm to (20.1, 5.60)
- moved R8 2.00 mm to (36.0, 8.28)
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Connections:
- net AGND: now also C_IN+12.C, C_IN+5.C, C_IN-12.A, C_IN-5.A; no longer C_IN+12.2, C_IN+5.2, C_IN-12.1, C_IN-5.1
- net N$1: now also C_IN-12.C, C_IN-5.C; no longer C_IN-12.2, C_IN-5.2
- net N$5: now also C_IN+12.A, C_IN+5.A; no longer C_IN+12.1, C_IN+5.1
Routing:
- net N$2: track 10.6 -> 18.4 mm
- net N$1: track 55.5 -> 48.8 mm
- net N$9: track 12.5 -> 19.1 mm, vias 0 -> 2
- net AGND: track 237.2 -> 232.0 mm, vias 2 -> 3
- net +-12_!ON!/OFF: track 97.6 -> 100.4 mm
- net N$10: track 21.3 -> 24.1 mm
- net N$5: track 81.1 -> 78.9 mm
- net N$7: track 23.2 -> 25.2 mm
- net N$11: track 6.14 -> 6.97 mm
- net N$4: track 5.70 -> 6.30 mm

Commit message: repaint power supply
Parts:
- J1: device SparkFun-Connectors:1X03_LONGPADS -> SparkFun-Connectors:1X04_LONGPADS
- moved J1 7.09 mm to (11.1, 27.4), turned to 180 degrees
- moved B2 2.33 mm to (4.60, 20.9)
- moved B1 2.24 mm to (4.74, 34.1)
Connections:
- removed net EXTGND: B1.~2, B2.~1, J1.2
- new net N$13: B1.~2, J1.3
- new net N$6: B2.~1, J1.2
- net AGND: now also B2.+; no longer B2.-
- net N$1: now also B2.-; no longer B2.+
- net ~15V_PLUS: now also J1.4; no longer J1.3
Routing:
- net AGND: track 232.0 -> 189.4 mm
- net EXTGND: track 15.2 -> 0.00 mm
- net N$1: track 48.8 -> 37.0 mm
- net ~15V_MINUS: track 3.01 -> 14.4 mm
- net N$6: track 0.00 -> 5.19 mm
- net N$13: track 0.00 -> 3.64 mm
- net N$5: track 78.9 -> 82.1 mm
- net ~15V_PLUS: track 3.05 -> 3.62 mm
- removed copper zone on layer 1, net AGND
- removed copper zone on layer 16, net AGND
Changed lines of the file:
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@@
 </autorouter>
 <elements>
-<element name="B1" library="rectifier" library_urn="urn:adsk.eagle:library:336" package="SOIC-4" value="MB6S" x="5.74" y="36.11"/>
-<element name="B2" library="rectifier" library_urn="urn:adsk.eagle:library:336" package="SOIC-4" value="MB6S" x="5.78" y="18.89" smashed="yes" rot="R180">
-<attribute name="NAME" x="1.905" y="15.02" size="1.27" layer="25" font="vector"/>
-<attribute name="VALUE" x="1.77" y="21.295" size="1.27" layer="27" font="vector" rot="R270"/>
-</element>
+<element name="B1" library="rectifier" library_urn="urn:adsk.eagle:library:336" package="SOIC-4" value="MB6S" x="4.74" y="34.11"/>
 <element name="C_IN+12" library="SparkFun-Passives" package="EIA3216" value="10uF" x="37.44" y="47.35" smashed="yes" rot="R180">
 <attribute name="NAME" x="39.98" y="45.969" size="0.4064" layer="25" rot="R180"/>
@@
 <attribute name="VALUE" x="42.588" y="19.435" size="0.8128" layer="27" rot="R90"/>
 </element>
-<element name="J1" library="SparkFun-Connectors" package="1X03_LONGPADS" value="" x="4.44" y="24.93" rot="R90"/>
+<element name="J1" library="SparkFun-Connectors" package="1X04_LONGPADS" value="" x="11.07" y="27.44" rot="R180">
+<attribute name="PROD_ID" value="CONN-09696" x="11.07" y="27.44" size="1.778" layer="27" rot="R180" display="off"/>
+</element>
 <element name="J2" library="SparkFun-Connectors" package="1X05_LONGPADS" value="" x="16.82" y="28.56" smashed="yes">
 <attribute name="NAME" x="15.55" y="30.592" size="0.6096" layer="25" font="vector" ratio="20"/>
@@
 <attribute name="VALUE" x="20.718" y="32.01" size="1" layer="21" font="vector"/>
 </element>
+<element name="B2" library="rectifier" library_urn="urn:adsk.eagle:library:336" package="SOIC-4" value="MB6S" x="4.6" y="20.9" rot="R180"/>
 </elements>
 <signals>
-<signal name="EXTGND">
-<contactref element="B2" pad="~1"/>
-<contactref element="B1" pad="~2"/>
-<contactref element="J1" pad="2"/>
-<wire x1="4.44" y1="27.47" x2="6.47" y2="27.47" width="1.016" layer="1"/>
-<wire x1="8" y1="29" x2="8" y2="31" width="1.016" layer="1"/>
-<wire x1="8" y1="31" x2="7" y2="32" width="1.016" layer="1"/>
-<wire x1="7" y1="32" x2="7.04" y2="32.04" width="1.016" layer="1"/>
-<wire x1="7.04" y1="32.04" x2="7.04" y2="33.06" width="1.016" layer="1"/>
-<wire x1="6.47" y1="27.47" x2="8" y2="29" width="1.016" layer="1"/>
-<wire x1="7.08" y1="21.94" x2="7.08" y2="23.08" width="1.016" layer="1"/>
-<wire x1="7.08" y1="23.08" x2="8" y2="24" width="1.016" layer="1"/>
-<wire x1="8" y1="24" x2="8" y2="25.94" width="1.016" layer="1"/>
-<wire x1="8" y1="25.94" x2="6.47" y2="27.47" width="1.016" layer="1"/>
-</signal>
-<signal name="~15V_MINUS">
-<contactref element="B2" pad="~2"/>
-<contactref element="J1" pad="1"/>
-<wire x1="4.48" y1="21.94" x2="4.44" y2="21.98" width="1.016" layer="1"/>
-<wire x1="4.44" y1="21.98" x2="4.44" y2="24.93" width="1.016" layer="1"/>
-</signal>
 <signal name="~15V_PLUS">
 <contactref element="B1" pad="~1"/>
-<contactref element="J1" pad="3"/>
-<wire x1="4.44" y1="33.06" x2="4.44" y2="30.01" width="1.016" layer="1"/>
+<contactref element="J1" pad="4"/>
+<wire x1="3.44" y1="31.06" x2="3.44" y2="27.45" width="1.27" layer="1"/>
+<wire x1="3.44" y1="27.45" x2="3.45" y2="27.44" width="1.27" layer="1"/>
 </signal>
 <signal name="N$5">
@@
 <contactref element="U4" pad="4"/>
 <contactref element="C_IN+5" pad="A"/>
-<wire x1="7.04" y1="39.16" x2="9.48" y2="41.6" width="1.016" layer="1"/>
-<wire x1="9.48" y1="41.6" x2="18.9" y2="41.6" width="1.016" layer="1"/>
+<wire x1="8.6" y1="41.6" x2="18.9" y2="41.6" width="1.016" layer="1"/>
 <wire x1="18.9" y1="41.6" x2="19.8582" y2="42.5582" width="1.016" layer="1"/>
 <wire x1="19.8582" y1="42.5582" x2="19.8582" y2="44.03" width="1.016" layer="1"/>
@@
 <wire x1="28" y1="43" x2="28" y2="51" width="2.54" layer="1"/>
 <wire x1="28" y1="51" x2="23" y2="56" width="2.54" layer="1"/>
-<wire x1="7.04" y1="39.16" x2="7.04" y2="39.96" width="1.016" layer="1"/>
-<wire x1="7.04" y1="39.96" x2="7" y2="40" width="1.016" layer="1"/>
+<wire x1="7" y1="40" x2="7.04" y2="39.96" width="1.016" layer="1"/>
+<wire x1="8.6" y1="41.6" x2="8" y2="41" width="1.016" layer="1"/>
+<wire x1="8" y1="41" x2="7" y2="40" width="1.016" layer="1"/>
+<wire x1="6.04" y1="37.16" x2="8.04" y2="40.96" width="2.54" layer="1"/>
+<wire x1="8.04" y1="40.96" x2="8" y2="41" width="2.54" layer="1"/>
 </signal>
 <signal name="AGND">
-<contactref element="B2" pad="-"/>
-<contactref element="B1" pad="-"/>
 <contactref element="R2" pad="1"/>
 <contactref element="R1" pad="1"/>
@@
 <wire x1="27.76" y1="38.14" x2="26.4618" y2="36.8418" width="1.016" layer="1"/>
 <wire x1="26.4618" y1="36.8418" x2="21.56" y2="36.8418" width="1.016" layer="1"/>
-<wire x1="13.17" y1="32.27" x2="10.73" y2="32.27" width="1.016" layer="1"/>
-<wire x1="9" y1="34" x2="9" y2="36" width="1.016" layer="1"/>
-<wire x1="9" y1="36" x2="5" y2="36" width="1.016" layer="1"/>
-<wire x1="5" y1="36" x2="4.44" y2="36.56" width="1.016" layer="1"/>
-<wire x1="4.44" y1="36.56" x2="4.44" y2="39.16" width="1.016" layer="1"/>
-<wire x1="10.73" y1="32.27" x2="9" y2="34" width="1.016" layer="1"/>
 <wire x1="21.9" y1="28.56" x2="21.9" y2="31.1" width="1.016" layer="16"/>
 <wire x1="20.73" y1="32.27" x2="13.17" y2="32.27" width="1.016" layer="16"/>
@@
 <wire x1="38.57" y1="24.41" x2="30.76" y2="32.22" width="1.016" layer="1"/>
 <wire x1="30.76" y1="32.22" x2="30.57" y2="32.22" width="1.016" layer="1"/>
-<wire x1="7.08" y1="15.84" x2="7.08" y2="16.92" width="1.016" layer="1"/>
-<polygon width="0.6096" layer="1">
-<vertex x="0" y="61"/>
-<vertex x="46" y="61"/>
-<vertex x="46" y="0"/>
-<vertex x="0" y="0"/>
-</polygon>
-<polygon width="0.6096" layer="16">
-<vertex x="0" y="61"/>
-<vertex x="46" y="61"/>
-<vertex x="46" y="0"/>
-<vertex x="0" y="0"/>
-</polygon>
 <wire x1="21.56" y1="44.03" x2="21.56" y2="47.02" width="1.016" layer="1"/>
 <wire x1="21.66" y1="47.12" x2="21.49" y2="47.25" width="1.016" layer="1"/>
@@
 <wire x1="34.92" y1="51.08" x2="33.44" y2="51.08" width="1.016" layer="1"/>
 <wire x1="36.36" y1="49.64" x2="34.92" y2="51.08" width="1.016" layer="1"/>
-<wire x1="4.44" y1="39.16" x2="4.44" y2="51.44" width="1.016" layer="1"/>
-<wire x1="4.44" y1="51.44" x2="5" y2="52" width="1.016" layer="1"/>
 <via x="5" y="52" extent="1-16" drill="0.35"/>
 <wire x1="5" y1="52" x2="8" y2="52" width="1.016" layer="16"/>
@@
 <wire x1="20.06" y1="4.7" x2="18.3" y2="4.7" width="1.016" layer="1"/>
 <wire x1="18.3" y1="4.7" x2="16.5" y2="6.5" width="1.016" layer="1"/>
-<wire x1="7.08" y1="16.92" x2="6" y2="18" width="1.016" layer="1"/>
-<wire x1="6" y1="18" x2="3" y2="18" width="1.016" layer="1"/>
-<wire x1="3" y1="18" x2="2" y2="17" width="1.016" layer="1"/>
-<wire x1="2" y1="17" x2="2" y2="14" width="1.016" layer="1"/>
-<wire x1="2" y1="14" x2="12" y2="4" width="1.016" layer="1"/>
-<wire x1="12" y1="4" x2="14" y2="4" width="1.016" layer="1"/>
-<wire x1="14" y1="4" x2="14.9" y2="4.9" width="1.016" layer="1"/>
-<wire x1="14.9" y1="4.9" x2="14.9" y2="6" width="1.016" layer="1"/>
 <wire x1="35.96" y1="4.37" x2="31.9" y2="4.37" width="1.016" layer="1"/>
 <wire x1="31.9" y1="4.37" x2="31.135" y2="5.135" width="1.016" layer="1"/>
@@
 <wire x1="38.58" y1="24.4" x2="38.57" y2="24.41" width="1.016" layer="1"/>
 <wire x1="39.6" y1="24.4" x2="38.58" y2="24.4" width="1.016" layer="1"/>
+<contactref element="B1" pad="-"/>
+<contactref element="B2" pad="+"/>
+<wire x1="13.17" y1="32.27" x2="10.73" y2="32.27" width="1.27" layer="1"/>
+<wire x1="10.73" y1="32.27" x2="9" y2="34" width="1.27" layer="1"/>
+<wire x1="9" y1="34" x2="4" y2="34" width="1.27" layer="1"/>
+<wire x1="4" y1="34" x2="3.44" y2="34.56" width="1.27" layer="1"/>
+<wire x1="3.44" y1="34.56" x2="3.44" y2="37.16" width="1.27" layer="1"/>
+<wire x1="39" y1="43.89" x2="38.86" y2="44.03" width="0" layer="19" extent="1-1"/>
+<wire x1="3.3" y1="17.85" x2="16.3818" y2="11.27" width="0" layer="19" extent="1-1"/>
 </signal>
 <signal name="+-12_!ON!/OFF">
@@
 <contactref element="U1" pad="3"/>
 <contactref element="U1" pad="TAB"/>
-<contactref element="B2" pad="+"/>
 <contactref element="C_IN-12" pad="C"/>
 <wire x1="30.58" y1="11.37" x2="30.58" y2="14" width="1.016" layer="1"/>
@@
 <wire x1="30.58" y1="11.37" x2="30.58" y2="8.08" width="1.016" layer="1"/>
 <wire x1="30.58" y1="8.08" x2="30.81" y2="7.85" width="1.016" layer="1"/>
-<wire x1="4.48" y1="15.84" x2="4.48" y2="14.52" width="1.016" layer="1"/>
-<wire x1="4.48" y1="14.52" x2="5" y2="14" width="1.016" layer="1"/>
-<wire x1="5" y1="14" x2="14.68" y2="14" width="1.016" layer="1"/>
 <wire x1="14.68" y1="14" x2="30.58" y2="14" width="1.016" layer="1"/>
+<contactref element="B2" pad="-"/>
+<wire x1="5.9" y1="17.85" x2="14.68" y2="11.27" width="0" layer="19" extent="1-1"/>
 </signal>
 <signal name="N$2">
@@
 <wire x1="20.8" y1="51.2" x2="19.9" y2="51.2" width="0.6096" layer="16"/>
 </signal>
+<signal name="~15V_MINUS">
+<contactref element="B2" pad="~2"/>
+<contactref element="J1" pad="1"/>
+<wire x1="3.3" y1="23.95" x2="3.3" y2="21.7" width="1.27" layer="1"/>
+<wire x1="3.3" y1="21.7" x2="4" y2="21" width="1.5" layer="1"/>
+<wire x1="4" y1="21" x2="7" y2="21" width="1.5" layer="1"/>
+<wire x1="11.07" y1="25.07" x2="11.07" y2="27.44" width="1.5" layer="1"/>
+<wire x1="7" y1="21" x2="11.07" y2="25.07" width="1.5" layer="1"/>
+</signal>
+<signal name="N$6">
+<contactref element="B2" pad="~1"/>
+<contactref element="J1" pad="2"/>
+<wire x1="5.9" y1="23.95" x2="5.95" y2="24" width="1.5" layer="1"/>
+<wire x1="5.95" y1="24" x2="7" y2="24" width="1.5" layer="1"/>
+<wire x1="7" y1="24" x2="8.53" y2="25.53" width="1.5" layer="1"/>
+<wire x1="8.53" y1="25.53" x2="8.53" y2="27.44" width="1.27" layer="1"/>
+</signal>
+<signal name="N$13">
+<contactref element="J1" pad="3"/>
+<contactref element="B1" pad="~2"/>
+<wire x1="6.04" y1="31.06" x2="6.04" y2="27.49" width="1.27" layer="1"/>
+<wire x1="6.04" y1="27.49" x2="5.99" y2="27.44" width="1.27" layer="1"/>
+</signal>
 </signals>

Commit message: minor changes
Routing:
- net AGND: track 189.4 -> 239.4 mm, vias 3 -> 4
- net N$1: track 37.0 -> 46.2 mm
- added copper zone on layer 1, net AGND
- added copper zone on layer 16, net AGND
Changed lines of the file:
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@@
 <drawing>
 <settings>
-<setting alwaysvectorfont="yes"/>
+<setting alwaysvectorfont="no"/>
 <setting verticaltext="up"/>
 </settings>
@@
 <contactref element="B1" pad="~1"/>
 <contactref element="J1" pad="4"/>
-<wire x1="3.44" y1="31.06" x2="3.44" y2="27.45" width="1.27" layer="1"/>
+<wire x1="3.44" y1="31.06" x2="3.44" y2="27.45" width="1.5" layer="1"/>
 <wire x1="3.44" y1="27.45" x2="3.45" y2="27.44" width="1.27" layer="1"/>
 </signal>
@@
 <contactref element="U4" pad="4"/>
 <contactref element="C_IN+5" pad="A"/>
-<wire x1="8.6" y1="41.6" x2="18.9" y2="41.6" width="1.016" layer="1"/>
-<wire x1="18.9" y1="41.6" x2="19.8582" y2="42.5582" width="1.016" layer="1"/>
+<wire x1="8.6" y1="41.6" x2="18.9" y2="41.6" width="1.5" layer="1"/>
+<wire x1="18.9" y1="41.6" x2="19.8582" y2="42.5582" width="1.5" layer="1"/>
 <wire x1="19.8582" y1="42.5582" x2="19.8582" y2="44.03" width="1.016" layer="1"/>
 <wire x1="37.1582" y1="44.03" x2="37.1582" y2="42.4582" width="1.016" layer="1"/>
-<wire x1="37.1582" y1="42.4582" x2="36.5" y2="41.8" width="1.016" layer="1"/>
-<wire x1="36.5" y1="41.8" x2="29.2" y2="41.8" width="1.016" layer="1"/>
+<wire x1="37.1582" y1="42.4582" x2="36.5" y2="41.8" width="1.5" layer="1"/>
+<wire x1="36.5" y1="41.8" x2="29.2" y2="41.8" width="1.5" layer="1"/>
 <wire x1="29.2" y1="41.8" x2="29" y2="42" width="1.016" layer="1"/>
 <wire x1="19.8582" y1="44.03" x2="19.8582" y2="46.3818" width="1.016" layer="1"/>
@@
 <wire x1="4" y1="34" x2="3.44" y2="34.56" width="1.27" layer="1"/>
 <wire x1="3.44" y1="34.56" x2="3.44" y2="37.16" width="1.27" layer="1"/>
+<wire x1="3.3" y1="17.85" x2="3.3" y2="11.7" width="1.5" layer="1"/>
+<wire x1="3.3" y1="11.7" x2="4.5" y2="10.5" width="1.5" layer="1"/>
+<wire x1="4.5" y1="10.5" x2="11" y2="4" width="1.5" layer="1"/>
+<wire x1="11" y1="4" x2="17.6" y2="4" width="1.5" layer="1"/>
+<wire x1="17.6" y1="4" x2="18.3" y2="4.7" width="1.5" layer="1"/>
+<wire x1="13.17" y1="32.27" x2="13.17" y2="19.17" width="1.5" layer="16"/>
+<wire x1="13.17" y1="19.17" x2="4.5" y2="10.5" width="1.5" layer="16"/>
+<via x="4.5" y="10.5" extent="1-16" drill="0.35"/>
+<polygon width="1.5" layer="16">
+<vertex x="0" y="61"/>
+<vertex x="46" y="61"/>
+<vertex x="46" y="0"/>
+<vertex x="0" y="0"/>
+</polygon>
+<polygon width="1.5" layer="1">
+<vertex x="0" y="61"/>
+<vertex x="46" y="61"/>
+<vertex x="46" y="0"/>
+<vertex x="0" y="0"/>
+</polygon>
 <wire x1="39" y1="43.89" x2="38.86" y2="44.03" width="0" layer="19" extent="1-1"/>
-<wire x1="3.3" y1="17.85" x2="16.3818" y2="11.27" width="0" layer="19" extent="1-1"/>
 </signal>
 <signal name="+-12_!ON!/OFF">
@@
 <wire x1="30.58" y1="14" x2="30.58" y2="18.5582" width="1.016" layer="1"/>
 <wire x1="14.68" y1="11.27" x2="14.68" y2="14" width="1.016" layer="1"/>
-<wire x1="14.68" y1="14" x2="14.68" y2="18.4582" width="1.016" layer="1"/>
+<wire x1="14.68" y1="14" x2="14.68" y2="17" width="1.016" layer="1"/>
+<wire x1="14.68" y1="17" x2="14.68" y2="18.4582" width="1.016" layer="1"/>
 <wire x1="30.5582" y1="18.5582" x2="30.58" y2="18.5582" width="1.016" layer="1"/>
 <wire x1="14.68" y1="18.34" x2="14.68" y2="18.4582" width="1.016" layer="1"/>
@@
 <wire x1="30.58" y1="11.37" x2="30.58" y2="8.08" width="1.016" layer="1"/>
 <wire x1="30.58" y1="8.08" x2="30.81" y2="7.85" width="1.016" layer="1"/>
-<wire x1="14.68" y1="14" x2="30.58" y2="14" width="1.016" layer="1"/>
+<wire x1="14.68" y1="14" x2="30.58" y2="14" width="1.5" layer="1"/>
 <contactref element="B2" pad="-"/>
-<wire x1="5.9" y1="17.85" x2="14.68" y2="11.27" width="0" layer="19" extent="1-1"/>
+<wire x1="5.9" y1="17.85" x2="13.83" y2="17.85" width="1.5" layer="1"/>
+<wire x1="13.83" y1="17.85" x2="14.68" y2="17" width="1.5" layer="1"/>
 </signal>
 <signal name="N$2">
@@
 <contactref element="B2" pad="~2"/>
 <contactref element="J1" pad="1"/>
-<wire x1="3.3" y1="23.95" x2="3.3" y2="21.7" width="1.27" layer="1"/>
+<wire x1="3.3" y1="23.95" x2="3.3" y2="21.7" width="1.5" layer="1"/>
 <wire x1="3.3" y1="21.7" x2="4" y2="21" width="1.5" layer="1"/>
 <wire x1="4" y1="21" x2="7" y2="21" width="1.5" layer="1"/>
@@
 <contactref element="J1" pad="3"/>
 <contactref element="B1" pad="~2"/>
-<wire x1="6.04" y1="31.06" x2="6.04" y2="27.49" width="1.27" layer="1"/>
+<wire x1="6.04" y1="31.06" x2="6.04" y2="27.49" width="1.5" layer="1"/>
 <wire x1="6.04" y1="27.49" x2="5.99" y2="27.44" width="1.27" layer="1"/>
 </signal>
