File: eagle/usb.brd (EAGLE design)
At the start: 160 x 100 mm, 45 parts, among them IC1 ICL7660CSA

Commit message: usb interface and dac were separated
Parts:
- removed C_OSC: (no value), SparkFun-Passives:1206
- removed I2S_CONVERTER:U$3: PCM1794A, EduAreaLib:SSOP28-0.65-10.2X5.2MM
- removed IC1: ICL7660CSA, maxim:SO08
- removed PCM2707-1:C1, PCM2707-1:C2, PCM2707-1:C5: 10uF, SparkFun-Passives:CPOL-RADIAL-100UF-25V
- removed PCM2707-1:C3, PCM2707-1:C4: 0.1uF, SparkFun-Passives:1206
- removed PCM2707-1:C6, PCM2707-1:C7: 1uF, SparkFun-Passives:1206
- removed PCM2707-1:J1: (no value), SparkFun-Connectors:1X04_LONGPADS
- removed PCM2707-1:R1, PCM2707-1:R6, PCM2707-1:R9: 1M, SparkFun-Passives:0805
- removed PCM2707-1:R2, PCM2707-1:R3: 22, SparkFun-Passives:0805
- removed PCM2707-1:R4: 400K, SparkFun-Passives:0805
- removed PCM2707-1:R5, PCM2707-1:R7, PCM2707-1:R8: 1.5K, SparkFun-Passives:0805
- removed PCM2707-1:U$1: PCM2707, EduAreaLib:TQFP32-0.8-7X7MM
- removed PCM2707-1:U$2: IRLML2246TRPBF, EduAreaLib:SOT23-3
- removed PCM2707-1:Y1: 12MHz CSTCE12MOG52-R0, SparkFun-Clocks:RESONATOR-SMD-3.2X1.3
- removed VR:B1, VR:B2: MB6S, rectifier:SOIC-4
- removed VR:C_IN+, VR:C_IN-, VR:C_OUT+, VR:C_OUT-: 10uF, SparkFun-Passives:EIA3216-KIT
- removed VR:J1, VR:J2: (no value), SparkFun-Connectors:1X03_LONGPADS
- removed VR:J3, VR:J4: (no value), SparkFun-Connectors:1X01
- removed VR:L1, VR:L2: (no value), SparkFun-Passives:INDUCTOR-1206
- removed VR:R1, VR:R2: 10K, SparkFun-Passives:0805
- removed VR:R3, VR:R5: 2.7K, SparkFun-Passives:0805
- removed VR:R4, VR:R6: ??, SparkFun-Passives:0805
- removed VR:U$1: LM2991, EduAreaLib:DDPAK/TO-263
- removed VR:U$2: LM2941, EduAreaLib:DDPAK/TO-263
- added C10, C11: 0.022uF, SparkFun-Passives:1206
- added C3, C4: 0.1uF, SparkFun-Passives:1206
- added C5: 10uF, SparkFun-Passives:CPOL-RADIAL-100UF-25V
- added C6, C7: 1uF, SparkFun-Passives:1206
- added C8, C9: 100uF, SparkFun-Passives:CPOL-RADIAL-100UF-25V
- added J1: (no value), SparkFun-Connectors:1X04_LONGPADS
- added J2: AUDIO_JACK_TRS_0.25"_PTH_RA, SparkFun-Connectors:AUDIO_JACK_0.25"_TRS_PTH_RA
- added J3: (no value), SparkFun-Connectors:1X04
- added J4: (no value), SparkFun-Connectors:MOLEX-1X6
- added J5: (no value), SparkFun-Connectors:1X02_LOCK_LONGPADS
- added R1, R6, R9: 1M, SparkFun-Passives:0805
- added R10, R11, R12, R13: 3.3K, SparkFun-Passives:0805
- added R14, R15: 16, SparkFun-Passives:0805
- added R2, R3: 22, SparkFun-Passives:0805
- added R4: 400K, SparkFun-Passives:0805
- added R5, R7, R8: 1.5K, SparkFun-Passives:0805
- added U$1: PCM2707, EduAreaLib:TQFP32-0.8-7X7MM
- added U$2: IRLML2246TRPBF, EduAreaLib:SOT23-3
- added Y1: 12MHz CSTCE12MOG52-R0, SparkFun-Clocks:RESONATOR-SMD-3.2X1.3
- C1, C2: value (none) -> 10uF; device SparkFun-Passives:EIA3216-KIT -> SparkFun-Passives:CPOL-RADIAL-100UF-25V
- moved C2 100.9 mm to (9.53, -62.5), turned to 0 degrees
- moved C1 61.7 mm to (35.9, -43.7), turned to 0 degrees
Connections:
- removed net +5V: C_OSC.2, IC1.8
- removed net -5V: C2.C, IC1.5
- removed net GND: C2.A, IC1.3
- removed net I2S_CONVERTER:BCK: I2S_CONVERTER:U$3.6
- removed net I2S_CONVERTER:DATA: I2S_CONVERTER:U$3.5
- removed net I2S_CONVERTER:LRCK: I2S_CONVERTER:U$3.4
- removed net I2S_CONVERTER:SCK: I2S_CONVERTER:U$3.7
- removed net PCM2707-1:!SUSPEND!: PCM2707-1:U$1.11
- removed net PCM2707-1:3.3V: PCM2707-1:C1.1, PCM2707-1:C2.1, PCM2707-1:C3.1, PCM2707-1:C4.1, PCM2707-1:C6.2, PCM2707-1:C7.1, PCM2707-1:R7.1, PCM2707-1:R8.2, PCM2707-1:U$1.2, PCM2707-1:U$1.21, PCM2707-1:U$1.27, PCM2707-1:U$1.30
- removed net PCM2707-1:BCK: PCM2707-1:U$1.19
- removed net PCM2707-1:DGND: PCM2707-1:C1.2, PCM2707-1:C2.2, PCM2707-1:C3.2, PCM2707-1:C4.2, PCM2707-1:C5.2, PCM2707-1:C6.1, PCM2707-1:C7.2, PCM2707-1:J1.4, PCM2707-1:R1.1, PCM2707-1:U$1.1, PCM2707-1:U$1.16, PCM2707-1:U$1.20, PCM2707-1:U$1.25, PCM2707-1:U$1.26, PCM2707-1:U$1.31, PCM2707-1:U$1.9, PCM2707-1:Y1.2
- removed net PCM2707-1:DIN: PCM2707-1:U$1.4
- removed net PCM2707-1:DOUT: PCM2707-1:U$1.17
- removed net PCM2707-1:LRCK: PCM2707-1:U$1.5
- removed net PCM2707-1:N$1: PCM2707-1:R6.1, PCM2707-1:U$1.12, PCM2707-1:Y1.1
- removed net PCM2707-1:N$2: PCM2707-1:R5.1, PCM2707-1:U$2.3
- removed net PCM2707-1:N$3: PCM2707-1:R6.2, PCM2707-1:U$1.13, PCM2707-1:Y1.3
- removed net PCM2707-1:N$4: PCM2707-1:R2.1, PCM2707-1:U$1.23
- removed net PCM2707-1:N$5: PCM2707-1:R3.1, PCM2707-1:U$1.22
- removed net PCM2707-1:N$6: PCM2707-1:C5.1, PCM2707-1:U$1.32
- removed net PCM2707-1:N$7: PCM2707-1:R7.2, PCM2707-1:U$1.15
- removed net PCM2707-1:N$8: PCM2707-1:R8.1, PCM2707-1:U$1.10
- removed net PCM2707-1:N$9: PCM2707-1:R9.2, PCM2707-1:U$1.3
- removed net PCM2707-1:PULLUP_HANDLE: PCM2707-1:R4.2, PCM2707-1:U$2.1
- removed net PCM2707-1:SPI_!SS!: PCM2707-1:U$1.6
- removed net PCM2707-1:SPI_CLCK: PCM2707-1:U$1.7
- removed net PCM2707-1:SPI_MOSI: PCM2707-1:U$1.8
- removed net PCM2707-1:SYSCK: PCM2707-1:U$1.18
- removed net PCM2707-1:USB_D+: PCM2707-1:J1.2, PCM2707-1:R2.2, PCM2707-1:R5.2
- removed net PCM2707-1:USB_D-: PCM2707-1:J1.3, PCM2707-1:R3.2
- removed net PCM2707-1:USB_VBUS: PCM2707-1:J1.1, PCM2707-1:R1.2, PCM2707-1:R4.1, PCM2707-1:R9.1, PCM2707-1:U$1.24, PCM2707-1:U$2.2
- removed net PCM2707-1:VOUT_L: PCM2707-1:U$1.28
- removed net PCM2707-1:VOUT_R: PCM2707-1:U$1.29
- removed net VR:!ON!/OFF: VR:J3.1, VR:R1.2, VR:R2.2, VR:U$1.2, VR:U$2.2
- removed net VR:+12V: VR:C_OUT+.A, VR:J2.1, VR:L2.P$2
- removed net VR:-12V: VR:C_OUT-.C, VR:J2.3, VR:L1.P$2
- removed net VR:AGND: VR:B1.-, VR:B2.-, VR:C_IN+.C, VR:C_IN-.A, VR:C_OUT+.C, VR:C_OUT-.A, VR:J2.2, VR:J4.1, VR:R1.1, VR:R2.1, VR:R4.1, VR:R6.1, VR:U$1.4, VR:U$2.3, VR:U$2.TAB
- removed net VR:EXTGND: VR:B1.~2, VR:B2.~1, VR:J1.2
- removed net VR:N$4: VR:L2.P$1, VR:R3.2, VR:U$2.5
- removed net VR:N$5: VR:B1.+, VR:C_IN+.A, VR:U$2.4
- removed net VR:N$6: VR:B2.+, VR:C_IN-.C, VR:U$1.3, VR:U$1.TAB
- removed net VR:N$7: VR:R3.1, VR:R4.2, VR:U$2.1
- removed net VR:N$8: VR:L1.P$1, VR:R5.2, VR:U$1.5
- removed net VR:N$9: VR:R5.1, VR:R6.2, VR:U$1.1
- removed net VR:~15V_MINUS: VR:B2.~2, VR:J1.1
- removed net VR:~15V_PLUS: VR:B1.~1, VR:J1.3
- new net !SUSPEND!: U$1.11
- new net 3.3V: C1.1, C2.1, C3.1, C4.1, C6.2, C7.1, J5.1, R7.1, R8.2, U$1.2, U$1.21, U$1.27, U$1.30
- new net BCK: J4.2, U$1.19
- new net DGND: C1.2, C2.2, C3.2, C4.2, C5.2, C6.1, C7.2, J1.4, R1.1, U$1.1, U$1.20, U$1.25, U$1.26, U$1.31, U$1.9, Y1.2
- new net DIN: J4.6, U$1.4
- new net DOUT: J4.4, U$1.17
- new net GNDA: J2.SLEEVE, J3.1, J4.1, J5.2, R10.2, R11.2, R12.2, R13.2, R14.2, R15.2, U$1.16
- new net LRCK: J4.5, U$1.5
- new net N$1: R6.1, U$1.12, Y1.1
- new net N$11: C9.2, J2.RING, R11.1
- new net N$14: C10.1, R14.1
- new net N$15: C11.1, R15.1
- new net N$4: R2.1, U$1.23
- new net N$5: R3.1, U$1.22
- new net N$6: C5.1, U$1.32
- new net N$7: R7.2, U$1.15
- new net N$8: R8.1, U$1.10
- new net N$9: R9.2, U$1.3
- new net PULLUP_HANDLE: R4.2, U$2.1
- new net SPI_!SS!: J3.2, U$1.6
- new net SPI_CLCK: J3.3, U$1.7
- new net SPI_MOSI: J3.4, U$1.8
- new net SYSCK: J4.3, U$1.18
- new net USB_D+: J1.2, R2.2, R5.2
- new net USB_D-: J1.3, R3.2
- new net USB_VBUS: J1.1, R1.2, R4.1, R9.1, U$1.24, U$2.2
- new net VOUT_L: C11.2, C8.1, R13.1, U$1.28
- new net VOUT_R: C10.2, C9.1, R12.1, U$1.29
- net N$10: now also C8.2, J2.TIP, R10.1; no longer C1.A, IC1.2
- net N$2: now also R5.1, U$2.3; no longer C_OSC.1, IC1.7
- net N$3: now also R6.2, U$1.13, Y1.3; no longer C1.C, IC1.4
Routing:
- net VR:AGND: track 124.2 -> 0.00 mm, vias 1 -> 0
- net VR:!ON!/OFF: track 32.3 -> 0.00 mm, vias 2 -> 0
- net VR:+12V: track 27.5 -> 0.00 mm
- net VR:-12V: track 25.9 -> 0.00 mm
- net VR:N$6: track 22.1 -> 0.00 mm
- net VR:N$4: track 21.3 -> 0.00 mm, vias 2 -> 0
- net VR:N$8: track 20.0 -> 0.00 mm, vias 2 -> 0
- net VR:N$5: track 16.0 -> 0.00 mm
- net VR:EXTGND: track 14.8 -> 0.00 mm
- net VR:~15V_MINUS: track 12.7 -> 0.00 mm
- net VR:~15V_PLUS: track 10.0 -> 0.00 mm
- net VR:N$9: track 8.31 -> 0.00 mm
- net VR:N$7: track 7.17 -> 0.00 mm
- net GND: track 6.13 -> 0.00 mm
- net -5V: track 4.43 -> 0.00 mm
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Other:
- board size 160 x 100 mm -> 80 x 61 mm

Commit message: usb interface and dac were separated
Parts:
- removed R4: 400K, SparkFun-Passives:0805
- removed U$2: IRLML2246TRPBF, EduAreaLib:SOT23-3
- added J6: (no value), SparkFun-Connectors:USB-AB-MICRO-SMD
- J1: device SparkFun-Connectors:1X04_LONGPADS -> SparkFun-Connectors:1X01
- moved J5 183.8 mm to (35.2, 37.5), turned to 270 degrees
- moved J4 157.2 mm to (35.1, 27.8), turned to 270 degrees
- moved R15 149.9 mm to (34.5, 50.8)
- moved R13 146.7 mm to (33.0, 55.2), turned to 90 degrees
- moved R10 145.7 mm to (30.5, 55.2), turned to 270 degrees
- moved J3 143.9 mm to (19.8, 36.7), turned to 180 degrees
- moved C11 141.5 mm to (29.7, 50.7), turned to 180 degrees
- moved R14 138.7 mm to (34.6, 46.8)
- moved C10 138.2 mm to (29.9, 46.9), turned to 180 degrees
- moved R12 133.7 mm to (33.0, 42.5), turned to 270 degrees
- moved R11 133.5 mm to (30.4, 42.5), turned to 90 degrees
- moved C9 122.8 mm to (25.4, 42.7)
- moved C8 119.1 mm to (25.6, 54.6)
- moved C3 111.1 mm to (20.8, 32.9)
- moved Y1 104.4 mm to (9.25, 24.9), turned to 270 degrees
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Connections:
- removed net N$2: R5.1, U$2.3
- removed net PULLUP_HANDLE: R4.2, U$2.1
- new net D+PULLPUP: J1.1, R5.1
- net DGND: now also J6.GND1; no longer J1.4
- net DOUT: now also J4.3; no longer J4.4
- net SYSCK: now also J4.4; no longer J4.3
- net USB_D+: now also J6.D+1; no longer J1.2
- net USB_D-: now also J6.D-1; no longer J1.3
- net USB_VBUS: now also J6.VBUS1; no longer J1.1, R4.1, U$2.2

Commit message: pre usb interface gamma
Parts:
- removed R9: 1M, SparkFun-Passives:0805
- added C12: 100uF, SparkFun-Passives:CPOL-RADIAL-100UF-25V
- added C13: 0.1uF, SparkFun-Passives:1206
- added J7: +5V, SparkFun-Connectors:1X02_LOCK_LONGPADS
- added J8: !SUSPND!, SparkFun-Connectors:1X01
- added U$2: LM3940IMP-3.3/NOPB, EduAreaLib:SOT223
- added U$3: (no value), EduAreaLib:CRIMEA_TOP
- J1: value (none) -> PULLUP
- J3: value (none) -> SPI
- J4: value (none) -> I2S
- J5: value (none) -> +3.3V
- J6: value (none) -> USB
- moved C6 55.3 mm to (11.0, 32.7)
- moved R8 52.9 mm to (11.4, 29.2), turned to 90 degrees
- moved C7 48.6 mm to (26.9, 26.1), turned to 90 degrees
- moved R6 46.9 mm to (10.9, 25.4), turned to 270 degrees
- moved R7 45.4 mm to (11.4, 22.3), turned to 90 degrees
- moved R1 37.9 mm to (8.53, 20.2), turned to 270 degrees
- moved R3 36.8 mm to (9.41, 17.7), turned to 180 degrees
- moved R5 36.5 mm to (9.39, 14.4), turned to 180 degrees
- moved R2 34.4 mm to (9.40, 16.1), turned to 180 degrees
- moved J1 16.1 mm to (7.82, 11.7)
- moved J4 11.3 mm to (34.9, 16.4), turned to 90 degrees
- moved C1 4.42 mm to (25.6, 16.4)
- moved C4 2.85 mm to (19.2, 16.9), turned to 180 degrees
- moved C2 2.57 mm to (14.5, 12.4), turned to 0 degrees
- moved C3 1.72 mm to (19.5, 34.1)
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Connections:
- removed net GNDA: J2.SLEEVE, J3.1, J4.1, J5.2, R10.2, R11.2, R12.2, R13.2, R14.2, R15.2, U$1.16
- removed net N$9: R9.2, U$1.3
- new net N$2: C13.2, J7.2, U$2.1
- net !SUSPEND!: now also J8.1
- net 3.3V: now also C12.1, U$2.3
- net DGND: now also C12.2, C13.1, J2.SLEEVE, J3.1, J4.1, J5.2, J7.1, R10.2, R11.2, R12.2, R13.2, R14.2, R15.2, U$1.16, U$2.2, U$2.4
- net DOUT: now also J4.4; no longer J4.3
- net SYSCK: now also J4.3; no longer J4.4
- net USB_VBUS: now also U$1.3; no longer R9.1
Routing:
- net DGND: track 0.00 -> 224.2 mm, vias 0 -> 4
- net 3.3V: track 0.00 -> 105.7 mm, vias 0 -> 6
- net USB_VBUS: track 0.00 -> 48.5 mm, vias 0 -> 4
- net VOUT_L: track 0.00 -> 43.6 mm, vias 0 -> 1
- net VOUT_R: track 0.00 -> 29.7 mm, vias 0 -> 1
- net N$2: track 0.00 -> 27.3 mm
- net N$10: track 0.00 -> 25.4 mm
- net N$11: track 0.00 -> 25.2 mm
- net DOUT: track 0.00 -> 24.7 mm, vias 0 -> 2
- net DIN: track 0.00 -> 24.1 mm, vias 0 -> 3
- net SYSCK: track 0.00 -> 22.9 mm, vias 0 -> 2
- net BCK: track 0.00 -> 22.3 mm, vias 0 -> 1
- net LRCK: track 0.00 -> 21.1 mm, vias 0 -> 2
- net N$4: track 0.00 -> 13.4 mm
- net N$5: track 0.00 -> 11.5 mm
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- added copper zone on layer 1, net DGND
- added copper zone on layer 16, net DGND
Other:
- board size 80 x 61 mm -> 38 x 61 mm

Commit message: beta usb interface
Parts:
- removed R8: 1.5K, SparkFun-Passives:0805
- removed U$2: LM3940IMP-3.3/NOPB, EduAreaLib:SOT223
- added FB1: (no value), SparkFun-Passives:1210
- added U2: LM3940IMP-3.3, EduAreaLib:SOT223
- J2: value AUDIO_JACK_TRS_0.25"_PTH_RA -> AUDIO_JACK_TRS_0.25"
- Y1: value 12MHz CSTCE12MOG52-R0 -> 12MHz
- moved C13 5.81 mm to (15.9, 4.94)
- moved J2 0.23 mm to (-0.02, 48.7)
- renumbered U$1 to UK1
Connections:
- removed net N$8: R8.1, UK1.10
- new net +5V: C13.2, J7.2, U2.1
- net 3.3V: now also FB1.2, UK1.10, UK1.24; no longer C12.1, R8.2, U$2.3
- net DGND: now also U2.2, U2.4; no longer U$2.2, U$2.4
- net N$2: now also C12.1, FB1.1, U2.3; no longer C13.2, J7.2, U$2.1
- net USB_VBUS: no longer UK1.24
Routing:
- net +5V: track 0.00 -> 20.5 mm
- net USB_VBUS: track 48.5 -> 31.5 mm, vias 4 -> 2
- net N$2: track 27.3 -> 11.2 mm
- net DGND: track 224.2 -> 229.9 mm
- net 3.3V: track 105.7 -> 110.4 mm, vias 6 -> 8
- net N$8: track 2.90 -> 0.00 mm
Other:
- board text added: "!SS!"
- board text added: "BCK"
- board text added: "CLCK"
- board text added: "DIN"
- board text added: "DOUT"
- board text added: "GND"
- board text added: "LRCK"
- board text added: "MOSI"
- board text added: "SYSCK"
