File: eagle/usb.sch (EAGLE design)
At the start: 4 parts, among them IC1 ICL7660CSA

Commit message: usb interface and dac were separated
Parts:
- removed C_OSC: (no value), SparkFun-Passives:CAP1206
- removed IC1: ICL7660CSA, maxim:ICL7660CSA
- added C10, C11: 0.022uF, SparkFun-Passives:CAP1206
- added C3, C4: 0.1uF, SparkFun-Passives:CAP1206
- added C5: 10uF, SparkFun-Passives:CAP_POLPTH1
- added C6, C7: 1uF, SparkFun-Passives:CAP1206
- added C8, C9: 100uF, SparkFun-Passives:CAP_POLPTH1
- added J1: (no value), SparkFun-Connectors:CONN_04LONGPADS
- added J2: AUDIO_JACK_TRS_0.25"_PTH_RA, SparkFun-Connectors:AUDIO_JACK_TRS_0.25"_PTH_RA
- added J3: (no value), SparkFun-Connectors:CONN_04
- added J4: (no value), SparkFun-Connectors:CONN_06POLAR
- added J5: (no value), SparkFun-Connectors:CONN_02LOCK_LONGPADS
- added R1, R6, R9: 1M, SparkFun-Passives:RESISTOR0805-RES
- added R10, R11, R12, R13: 3.3K, SparkFun-Passives:RESISTOR0805-RES
- added R14, R15: 16, SparkFun-Passives:RESISTOR0805-RES
- added R2, R3: 22, SparkFun-Passives:RESISTOR0805-RES
- added R4: 400K, SparkFun-Passives:RESISTOR0805-RES
- added R5, R7, R8: 1.5K, SparkFun-Passives:RESISTOR0805-RES
- added U$1: PCM2707, EduAreaLib:PCM2707
- added U$2: IRLML2246TRPBF, EduAreaLib:IRLML2246TRPBF
- added Y1: 12MHz CSTCE12MOG52-R0, SparkFun-Clocks:RESONATORSMD-3.2X1.3
- C1, C2: value (none) -> 10uF; device SparkFun-Passives:CAP_POL1206-KIT -> SparkFun-Passives:CAP_POLPTH1
Connections:
- removed net +5V: C_OSC.2, IC1.V+
- removed net -5V: C2.-, IC1.VOUT
- removed net 5V: C1.+
- removed net AGND: C1.-
- removed net GND: C2.+, IC1.GND
- new net !SUSPEND!: U$1.!SSPND!
- new net BCK: J4.2, U$1.FUNC1
- new net DIN: J4.6, U$1.FUNC3
- new net DOUT: J4.4, U$1.DOUT
- new net GNDA: J2.EARTH, J3.1, J4.1, J5.2, R10.2, R11.2, R12.2, R13.2, R14.2, R15.2, U$1.PSEL
- new net LRCK: J4.5, U$1.FUNC0
- new net N$1: R6.1, U$1.XTI, Y1.1
- new net N$11: C9.-, J2.RING, R11.1
- new net N$14: C10.1, R14.1
- new net N$15: C11.1, R15.1
- new net N$4: R2.1, U$1.D+
- new net N$5: R3.1, U$1.D-
- new net N$6: C5.+, U$1.VCOM
- new net N$7: R7.2, U$1.DT
- new net N$8: R8.1, U$1.TEST
- new net N$9: R9.2, U$1.HOST
- new net PULLUP_HANDLE: R4.2, U$2.G
- new net SPI_!SS!: J3.2, U$1.HID0/MS
- new net SPI_CLCK: J3.3, U$1.HID1/MC
- new net SPI_MOSI: J3.4, U$1.HID2/MD
- new net SYSCK: J4.3, U$1.FUNC2
- new net USB_D+: J1.2, R2.2, R5.2
- new net USB_D-: J1.3, R3.2
- new net USB_VBUS: J1.1, R1.2, R4.1, R9.1, U$1.VBUS, U$2.S
- new net VOUT_L: C11.2, C8.+, R13.1, U$1.VOUTL
- new net VOUT_R: C10.2, C9.+, R12.1, U$1.VOUTR
- net 3.3V: now also C3.1, C4.1, C6.2, C7.1, J5.1, R7.1, R8.2, U$1.VCCL, U$1.VCCP, U$1.VCCR, U$1.VDD
- net DGND: now also C3.2, C4.2, C5.-, C6.1, C7.2, J1.4, R1.1, U$1.AGNDL, U$1.AGNDR, U$1.DGND, U$1.FSEL, U$1.PGND, U$1.ZGND, Y1.2
- net N$10: now also C8.-, J2.TIP, R10.1; no longer C1.+, IC1.CAP+
- net N$2: now also R5.1, U$2.D; no longer C_OSC.1, IC1.OSC
- net N$3: now also R6.2, U$1.XTO, Y1.3; no longer C1.-, IC1.CAP-
Other:
- note removed: "AC-DC converter +-12-15V"

Commit message: usb interface and dac were separated
Parts:
- removed R4: 400K, SparkFun-Passives:RESISTOR0805-RES
- removed U$2: IRLML2246TRPBF, EduAreaLib:IRLML2246TRPBF
- added J6: (no value), SparkFun-Connectors:USB_AB_SMT
- J1: device SparkFun-Connectors:CONN_04LONGPADS -> SparkFun-Connectors:CONN_01
Connections:
- removed net N$2: R5.1, U$2.D
- removed net PULLUP_HANDLE: R4.2, U$2.G
- new net D+PULLPUP: J1.1, R5.1
- net DGND: now also J6.GND; no longer J1.4
- net DOUT: now also J4.3; no longer J4.4
- net SYSCK: now also J4.4; no longer J4.3
- net USB_D+: now also J6.D+; no longer J1.2
- net USB_D-: now also J6.D-; no longer J1.3
- net USB_VBUS: now also J6.VBUS; no longer J1.1, R4.1, U$2.S
Changed lines of the file:
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@@
 <attribute name="SPICEPREFIX" value="U"/>
 </part>
-<part name="J1" library="SparkFun-Connectors" deviceset="CONN_04" device="LONGPADS"/>
 <part name="R1" library="SparkFun-Passives" deviceset="RESISTOR" device="0805-RES" value="1M"/>
 <part name="GND2" library="supply1" library_urn="urn:adsk.eagle:library:371" deviceset="GNDA" device="" value="GND"/>
 <part name="R2" library="SparkFun-Passives" deviceset="RESISTOR" device="0805-RES" value="22"/>
 <part name="R3" library="SparkFun-Passives" deviceset="RESISTOR" device="0805-RES" value="22"/>
-<part name="GND3" library="supply1" library_urn="urn:adsk.eagle:library:371" deviceset="GNDA" device="" value="GND"/>
 <part name="SUPPLY1" library="SparkFun-PowerSymbols" deviceset="3.3V" device=""/>
 <part name="GND4" library="supply1" library_urn="urn:adsk.eagle:library:371" deviceset="GNDA" device="" value="GND"/>
-<part name="U$2" library="EduAreaLib" deviceset="IRLML2246TRPBF" device=""/>
-<part name="R4" library="SparkFun-Passives" deviceset="RESISTOR" device="0805-RES" value="400K"/>
 <part name="GND5" library="supply1" library_urn="urn:adsk.eagle:library:371" deviceset="GNDA" device="" value="GND"/>
 <part name="R5" library="SparkFun-Passives" deviceset="RESISTOR" device="0805-RES" value="1.5K"/>
@@
 <part name="GND17" library="supply1" library_urn="urn:adsk.eagle:library:371" deviceset="GNDA" device="" value="GND"/>
 <part name="SUPPLY6" library="SparkFun-PowerSymbols" deviceset="3.3V" device=""/>
+<part name="J6" library="SparkFun-Connectors" deviceset="USB_AB" device="_SMT"/>
+<part name="GND18" library="supply1" library_urn="urn:adsk.eagle:library:371" deviceset="GNDA" device="" value="GND"/>
+<part name="J1" library="SparkFun-Connectors" deviceset="CONN_01" device=""/>
 </parts>
 <sheets>
@@
 </instance>
 <instance part="U$1" gate="G$1" x="180.34" y="88.9"/>
-<instance part="J1" gate="G$1" x="139.7" y="129.54"/>
 <instance part="R1" gate="G$1" x="160.02" y="119.38" rot="R90"/>
 <instance part="GND2" gate="1" x="160.02" y="109.22"/>
 <instance part="R2" gate="G$1" x="170.18" y="129.54" rot="R180"/>
 <instance part="R3" gate="G$1" x="160.02" y="132.08" rot="R180"/>
-<instance part="GND3" gate="1" x="152.4" y="139.7"/>
 <instance part="SUPPLY1" gate="G$1" x="180.34" y="152.4"/>
 <instance part="GND4" gate="1" x="190.5" y="129.54"/>
-<instance part="U$2" gate="G$1" x="149.86" y="160.02"/>
-<instance part="R4" gate="G$1" x="137.16" y="160.02" rot="R90"/>
 <instance part="GND5" gate="1" x="208.28" y="76.2"/>
 <instance part="R5" gate="G$1" x="165.1" y="147.32" rot="R270"/>
@@
 <instance part="GND17" gate="1" x="233.68" y="142.24"/>
 <instance part="SUPPLY6" gate="G$1" x="223.52" y="152.4"/>
+<instance part="J6" gate="G$1" x="101.6" y="129.54" rot="R180"/>
+<instance part="GND18" gate="1" x="109.22" y="121.92"/>
+<instance part="J1" gate="G$1" x="154.94" y="160.02"/>
 </instances>
 <busses>
@@
 <junction x="149.86" y="101.6"/>
 <junction x="154.94" y="101.6"/>
-</segment>
-<segment>
-<pinref part="J1" gate="G$1" pin="4"/>
-<wire x1="144.78" y1="134.62" x2="144.78" y2="144.78" width="0.1524" layer="91"/>
-<wire x1="144.78" y1="144.78" x2="152.4" y2="144.78" width="0.1524" layer="91"/>
-<pinref part="GND3" gate="1" pin="GNDA"/>
-<wire x1="152.4" y1="144.78" x2="152.4" y2="142.24" width="0.1524" layer="91"/>
-<label x="132.08" y="134.62" size="1.778" layer="95" rot="R180"/>
 </segment>
 <segment>
@@
 <junction x="149.86" y="66.04"/>
 </segment>
+<segment>
+<pinref part="J6" gate="G$1" pin="GND"/>
+<wire x1="106.68" y1="124.46" x2="109.22" y2="124.46" width="0.1524" layer="91"/>
+<pinref part="GND18" gate="1" pin="GNDA"/>
+<label x="111.76" y="124.46" size="1.778" layer="95"/>
+</segment>
 </net>
 <net name="USB_VBUS" class="0">
@@
 <pinref part="U$1" gate="G$1" pin="VBUS"/>
 <wire x1="172.72" y1="114.3" x2="172.72" y2="127" width="0.1524" layer="91"/>
-<pinref part="J1" gate="G$1" pin="1"/>
 <wire x1="172.72" y1="127" x2="160.02" y2="127" width="0.1524" layer="91"/>
 <pinref part="R1" gate="G$1" pin="2"/>
@@
 <wire x1="160.02" y1="127" x2="160.02" y2="124.46" width="0.1524" layer="91"/>
 <junction x="160.02" y="127"/>
-<label x="132.08" y="127" size="1.778" layer="95" rot="R180"/>
-</segment>
-<segment>
-<pinref part="U$2" gate="G$1" pin="S"/>
-<wire x1="139.7" y1="152.4" x2="137.16" y2="152.4" width="0.1524" layer="91"/>
-<pinref part="R4" gate="G$1" pin="1"/>
-<wire x1="137.16" y1="152.4" x2="137.16" y2="154.94" width="0.1524" layer="91"/>
-<wire x1="137.16" y1="152.4" x2="129.54" y2="152.4" width="0.1524" layer="91"/>
-<junction x="137.16" y="152.4"/>
-<label x="127" y="152.4" size="1.778" layer="95" rot="R180"/>
 </segment>
 <segment>
@@
 <wire x1="177.8" y1="48.26" x2="177.8" y2="45.72" width="0.1524" layer="91"/>
 </segment>
+<segment>
+<pinref part="J6" gate="G$1" pin="VBUS"/>
+<wire x1="106.68" y1="134.62" x2="109.22" y2="134.62" width="0.1524" layer="91"/>
+<label x="111.76" y="134.62" size="1.778" layer="95"/>
+</segment>
 </net>
 <net name="USB_D-" class="0">
 <segment>
 <pinref part="R3" gate="G$1" pin="2"/>
-<pinref part="J1" gate="G$1" pin="3"/>
 <wire x1="154.94" y1="132.08" x2="144.78" y2="132.08" width="0.1524" layer="91"/>
-<label x="132.08" y="132.08" size="1.778" layer="95" rot="R180"/>
+</segment>
+<segment>
+<pinref part="J6" gate="G$1" pin="D-"/>
+<wire x1="106.68" y1="132.08" x2="109.22" y2="132.08" width="0.1524" layer="91"/>
+<label x="109.22" y="132.08" size="1.778" layer="95"/>
 </segment>
 </net>
 <net name="USB_D+" class="0">
 <segment>
-<pinref part="J1" gate="G$1" pin="2"/>
 <pinref part="R2" gate="G$1" pin="2"/>
 <wire x1="144.78" y1="129.54" x2="165.1" y2="129.54" width="0.1524" layer="91"/>
-<label x="132.08" y="129.54" size="1.778" layer="95" rot="R180"/>
 <pinref part="R5" gate="G$1" pin="2"/>
 <wire x1="165.1" y1="129.54" x2="165.1" y2="142.24" width="0.1524" layer="91"/>
 <junction x="165.1" y="129.54"/>
+</segment>
+<segment>
+<pinref part="J6" gate="G$1" pin="D+"/>
+<wire x1="106.68" y1="129.54" x2="109.22" y2="129.54" width="0.1524" layer="91"/>
+<label x="109.22" y="129.54" size="1.778" layer="95"/>
 </segment>
 </net>
@@
 </segment>
 </net>
-<net name="PULLUP_HANDLE" class="0">
-<segment>
-<pinref part="U$2" gate="G$1" pin="G"/>
-<wire x1="139.7" y1="167.64" x2="137.16" y2="167.64" width="0.1524" layer="91"/>
-<pinref part="R4" gate="G$1" pin="2"/>
-<wire x1="137.16" y1="167.64" x2="129.54" y2="167.64" width="0.1524" layer="91"/>
-<wire x1="137.16" y1="165.1" x2="137.16" y2="167.64" width="0.1524" layer="91"/>
-<junction x="137.16" y="167.64"/>
-<label x="129.54" y="167.64" size="1.778" layer="95" rot="R180" xref="yes"/>
-</segment>
-</net>
-<net name="N$2" class="0">
-<segment>
-<pinref part="U$2" gate="G$1" pin="D"/>
+<net name="D+PULLPUP" class="0">
+<segment>
 <wire x1="165.1" y1="160.02" x2="162.56" y2="160.02" width="0.1524" layer="91"/>
 <pinref part="R5" gate="G$1" pin="1"/>
 <wire x1="165.1" y1="160.02" x2="165.1" y2="152.4" width="0.1524" layer="91"/>
+<pinref part="J1" gate="G$1" pin="1"/>
+<label x="165.1" y="160.02" size="1.778" layer="95"/>
 </segment>
 </net>
@@
 </segment>
 <segment>
-<pinref part="J4" gate="G$1" pin="4"/>
-<wire x1="127" y1="30.48" x2="134.62" y2="30.48" width="0.1524" layer="91"/>
-<label x="134.62" y="30.48" size="1.778" layer="95"/>
+<pinref part="J4" gate="G$1" pin="3"/>
+<wire x1="127" y1="27.94" x2="134.62" y2="27.94" width="0.1524" layer="91"/>
+<label x="134.62" y="27.94" size="1.778" layer="95"/>
 </segment>
 </net>
@@
 </segment>
 <segment>
-<pinref part="J4" gate="G$1" pin="3"/>
-<wire x1="127" y1="27.94" x2="134.62" y2="27.94" width="0.1524" layer="91"/>
-<label x="134.62" y="27.94" size="1.778" layer="95"/>
-</segment>
-</net>
+<pinref part="J4" gate="G$1" pin="4"/>
+<wire x1="127" y1="30.48" x2="134.62" y2="30.48" width="0.1524" layer="91"/>
+<label x="134.62" y="30.48" size="1.778" layer="95"/>
+</segment>
+</net>

Commit message: pre usb interface gamma
Parts:
- removed R9: 1M, SparkFun-Passives:RESISTOR0805-RES
- added C12: 100uF, SparkFun-Passives:CAP_POLPTH1
- added C13: 0.1uF, SparkFun-Passives:CAP1206
- added J7: +5V, SparkFun-Connectors:CONN_02LOCK_LONGPADS
- added J8: !SUSPND!, SparkFun-Connectors:CONN_01
- added U$2: LM3940IMP-3.3/NOPB, EduAreaLib:LM3940IMP-3.3/NOPB
- J1: value (none) -> PULLUP
- J3: value (none) -> SPI
- J4: value (none) -> I2S
- J5: value (none) -> +3.3V
- J6: value (none) -> USB
Connections:
- removed net GNDA: J2.EARTH, J3.1, J4.1, J5.2, R10.2, R11.2, R12.2, R13.2, R14.2, R15.2, U$1.PSEL
- removed net N$9: R9.2, U$1.HOST
- new net N$2: C13.2, J7.2, U$2.IN
- net !SUSPEND!: now also J8.1
- net 3.3V: now also C12.+, U$2.OUT
- net DGND: now also C12.-, C13.1, J2.EARTH, J3.1, J4.1, J5.2, J7.1, R10.2, R11.2, R12.2, R13.2, R14.2, R15.2, U$1.PSEL, U$2.GND
- net DOUT: now also J4.4; no longer J4.3
- net SYSCK: now also J4.3; no longer J4.4
- net USB_VBUS: now also U$1.HOST; no longer R9.1
Other:
- moved on the sheet: R3

Commit message: beta usb interface
Parts:
- removed R8: 1.5K, SparkFun-Passives:RESISTOR0805-RES
- added FB1: (no value), SparkFun-Passives:INDUCTOR1210
- J2: value AUDIO_JACK_TRS_0.25"_PTH_RA -> AUDIO_JACK_TRS_0.25"
- U2: value LM3940IMP-3.3/NOPB -> LM3940IMP-3.3
- Y1: value 12MHz CSTCE12MOG52-R0 -> 12MHz
- renumbered U$1 to UK1, U$2 to U2
Connections:
- net N$2 renamed +5V
- removed net N$8: R8.1, UK1.TEST
- new net N$2: C12.+, FB1.1, U2.OUT
- net 3.3V: now also FB1.2, UK1.TEST, UK1.VBUS; no longer C12.+, R8.2, U2.OUT
- net USB_VBUS: no longer UK1.VBUS
Other:
- moved on the sheet: R1
