File: eagle/dac.brd (EAGLE design)
At the start: 160 x 100 mm, 51 parts, among them IC1 ICL7660CSA

Commit message: usb interface and dac were separated
Parts:
- removed C1, C2: (no value), SparkFun-Passives:EIA3216-KIT
- removed C_OSC: (no value), SparkFun-Passives:1206
- removed IC1: ICL7660CSA, maxim:SO08
- removed VR:B1, VR:B2: MB6S, rectifier:SOIC-4
- removed VR:C_IN+, VR:C_IN-, VR:C_OUT+, VR:C_OUT-: 10uF, SparkFun-Passives:EIA3216-KIT
- removed VR:J1, VR:J2: (no value), SparkFun-Connectors:1X03_LONGPADS
- removed VR:J3, VR:J4: (no value), SparkFun-Connectors:1X01
- removed VR:L1, VR:L2: (no value), SparkFun-Passives:INDUCTOR-1206
- removed VR:R1, VR:R2: 10K, SparkFun-Passives:0805
- removed VR:R3, VR:R5: 2.7K, SparkFun-Passives:0805
- removed VR:R4, VR:R6: ??, SparkFun-Passives:0805
- removed VR:U$1: LM2991, EduAreaLib:DDPAK/TO-263
- removed VR:U$2: LM2941, EduAreaLib:DDPAK/TO-263
- added DAC1:C10, DAC1:C12, DAC1:C19, DAC1:C20, DAC1:C9: 10uF, SparkFun-Passives:CPOL-RADIAL-100UF-25V
- added DAC1:C11, DAC1:C13, DAC1:C22, DAC1:C23: 0.1uF, SparkFun-Passives:1206
- added DAC1:C14, DAC1:C15, DAC1:C16, DAC1:C17: 2.7nF, SparkFun-Passives:1206
- added DAC1:C18, DAC1:C21, PCM2707-1:C8, PCM2707-1:C9: 100uF, SparkFun-Passives:CPOL-RADIAL-100UF-25V
- added DAC1:C7, DAC1:C8: 47uF, SparkFun-Passives:CPOL-RADIAL-100UF-25V
- added DAC1:IC1: OPA4134UA, linear:SO14
- added DAC1:R1: 10K, SparkFun-Passives:0805
- added DAC1:R10, DAC1:R11, DAC1:R12, DAC1:R2, DAC1:R3, DAC1:R4, DAC1:R5, DAC1:R6, DAC1:R7, DAC1:R8: 1K, SparkFun-Passives:0805
- added DAC1:R13, DAC1:R9: 39.2, SparkFun-Passives:0805
- added DAC1:U$6: TPA6120A2, EduAreaLib:SOIC20S
- added PCM2707-1:C10, PCM2707-1:C11: 0.022uF, SparkFun-Passives:1206
- added PCM2707-1:J2: AUDIO_JACK_TRS_0.25"_PTH_RA, SparkFun-Connectors:AUDIO_JACK_0.25"_TRS_PTH_RA
- added PCM2707-1:R10, PCM2707-1:R11, PCM2707-1:R12, PCM2707-1:R13: 3.3K, SparkFun-Passives:0805
- added PCM2707-1:R14, PCM2707-1:R15: 16, SparkFun-Passives:0805
Connections:
- removed net +5V: C_OSC.2, IC1.8
- removed net -5V: C2.C, IC1.5
- removed net GND: C2.A, IC1.3
- removed net N$10: C1.A, IC1.2
- removed net N$2: C_OSC.1, IC1.7
- removed net N$3: C1.C, IC1.4
- removed net VR:!ON!/OFF: VR:J3.1, VR:R1.2, VR:R2.2, VR:U$1.2, VR:U$2.2
- removed net VR:+12V: VR:C_OUT+.A, VR:J2.1, VR:L2.P$2
- removed net VR:-12V: VR:C_OUT-.C, VR:J2.3, VR:L1.P$2
- removed net VR:AGND: VR:B1.-, VR:B2.-, VR:C_IN+.C, VR:C_IN-.A, VR:C_OUT+.C, VR:C_OUT-.A, VR:J2.2, VR:J4.1, VR:R1.1, VR:R2.1, VR:R4.1, VR:R6.1, VR:U$1.4, VR:U$2.3, VR:U$2.TAB
- removed net VR:EXTGND: VR:B1.~2, VR:B2.~1, VR:J1.2
- removed net VR:N$4: VR:L2.P$1, VR:R3.2, VR:U$2.5
- removed net VR:N$5: VR:B1.+, VR:C_IN+.A, VR:U$2.4
- removed net VR:N$6: VR:B2.+, VR:C_IN-.C, VR:U$1.3, VR:U$1.TAB
- removed net VR:N$7: VR:R3.1, VR:R4.2, VR:U$2.1
- removed net VR:N$8: VR:L1.P$1, VR:R5.2, VR:U$1.5
- removed net VR:N$9: VR:R5.1, VR:R6.2, VR:U$1.1
- removed net VR:~15V_MINUS: VR:B2.~2, VR:J1.1
- removed net VR:~15V_PLUS: VR:B1.~1, VR:J1.3
- new net DAC1:+12V: DAC1:C10.1, DAC1:C11.2, DAC1:C18.1, DAC1:C19.1, DAC1:C22.1, DAC1:IC1.4, DAC1:U$6.18, DAC1:U$6.3
- new net DAC1:-12V: DAC1:C12.2, DAC1:C13.2, DAC1:C20.2, DAC1:C21.2, DAC1:C23.1, DAC1:IC1.11, DAC1:U$6.1, DAC1:U$6.20
- new net DAC1:LOUT: DAC1:R9.2
- new net DAC1:N$1: DAC1:C14.2, DAC1:IC1.2, DAC1:R2.1, DAC1:U$1.26
- new net DAC1:N$10: DAC1:R10.2, DAC1:R11.2, DAC1:U$6.17
- new net DAC1:N$11: DAC1:R12.2, DAC1:R13.1, DAC1:U$6.19
- new net DAC1:N$14: DAC1:C15.1, DAC1:IC1.7, DAC1:R3.2, DAC1:R6.1
- new net DAC1:N$17: DAC1:C16.2, DAC1:IC1.9, DAC1:R4.1, DAC1:U$1.18
- new net DAC1:N$2: DAC1:C15.2, DAC1:IC1.6, DAC1:R3.1, DAC1:U$1.25
- new net DAC1:N$20: DAC1:C16.1, DAC1:IC1.8, DAC1:R12.1, DAC1:R4.2, DAC1:U$6.16
- new net DAC1:N$23: DAC1:C17.2, DAC1:IC1.13, DAC1:R5.1, DAC1:U$1.17
- new net DAC1:N$25: DAC1:C17.1, DAC1:IC1.14, DAC1:R11.1, DAC1:R5.2
- new net DAC1:N$3: DAC1:R1.1, DAC1:U$1.20
- new net DAC1:N$4: DAC1:R6.2, DAC1:R7.2, DAC1:U$6.4
- new net DAC1:N$5: DAC1:C7.2, DAC1:U$1.22
- new net DAC1:N$6: DAC1:C8.2, DAC1:U$1.21
- new net DAC1:N$8: DAC1:C14.1, DAC1:IC1.1, DAC1:R2.2, DAC1:R8.1, DAC1:U$6.5
- new net DAC1:N$9: DAC1:R8.2, DAC1:R9.1, DAC1:U$6.2
- new net DAC1:ROUT: DAC1:R13.2
- new net PCM2707-1:GNDA: PCM2707-1:J2.SLEEVE, PCM2707-1:R10.2, PCM2707-1:R11.2, PCM2707-1:R12.2, PCM2707-1:R13.2, PCM2707-1:R14.2, PCM2707-1:R15.2, PCM2707-1:U$1.16
- new net PCM2707-1:N$10: PCM2707-1:C8.2, PCM2707-1:J2.TIP, PCM2707-1:R10.1
- new net PCM2707-1:N$11: PCM2707-1:C9.2, PCM2707-1:J2.RING, PCM2707-1:R11.1
- new net PCM2707-1:N$14: PCM2707-1:C10.1, PCM2707-1:R14.1
- new net PCM2707-1:N$15: PCM2707-1:C11.1, PCM2707-1:R15.1
- net DAC1:3.3V: now also DAC1:C10.2, DAC1:C11.1, DAC1:C12.1, DAC1:C13.1, DAC1:IC1.10, DAC1:IC1.12, DAC1:IC1.3, DAC1:IC1.5, DAC1:R10.1, DAC1:R7.1
- net DAC1:5V: now also DAC1:C7.1, DAC1:C8.1, DAC1:C9.1, DAC1:U$1.23
- net DAC1:AGND: now also DAC1:C18.2, DAC1:C19.2, DAC1:C20.1, DAC1:C21.1, DAC1:C22.2, DAC1:C23.2, DAC1:C9.2, DAC1:R1.2, DAC1:U$1.19, DAC1:U$1.24
- net PCM2707-1:DGND: no longer PCM2707-1:U$1.16
- net PCM2707-1:VOUT_L: now also PCM2707-1:C11.2, PCM2707-1:C8.1, PCM2707-1:R13.1
- net PCM2707-1:VOUT_R: now also PCM2707-1:C10.2, PCM2707-1:C9.1, PCM2707-1:R12.1
Routing:
- net VR:AGND: track 124.2 -> 0.00 mm, vias 1 -> 0
- net VR:!ON!/OFF: track 32.3 -> 0.00 mm, vias 2 -> 0
- net VR:+12V: track 27.5 -> 0.00 mm
- net VR:-12V: track 25.9 -> 0.00 mm
- net VR:N$6: track 22.1 -> 0.00 mm
- net VR:N$4: track 21.3 -> 0.00 mm, vias 2 -> 0
- net VR:N$8: track 20.0 -> 0.00 mm, vias 2 -> 0
- net VR:N$5: track 16.0 -> 0.00 mm
- net VR:EXTGND: track 14.8 -> 0.00 mm
- net VR:~15V_MINUS: track 12.7 -> 0.00 mm
- net VR:~15V_PLUS: track 10.0 -> 0.00 mm
- net VR:N$9: track 8.31 -> 0.00 mm
- net VR:N$7: track 7.17 -> 0.00 mm
- net GND: track 6.13 -> 0.00 mm
- net -5V: track 4.43 -> 0.00 mm
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
Commit message: some minor changes
Parts:
- removed DAC1:C1, DAC1:C10, DAC1:C12, DAC1:C19, DAC1:C2, DAC1:C20, DAC1:C6, DAC1:C9, PCM2707-1:C1, PCM2707-1:C2, PCM2707-1:C5: 10uF, SparkFun-Passives:CPOL-RADIAL-100UF-25V
- removed DAC1:C11, DAC1:C13, DAC1:C22, DAC1:C23, DAC1:C3, DAC1:C4, DAC1:C5, PCM2707-1:C3, PCM2707-1:C4: 0.1uF, SparkFun-Passives:1206
- removed DAC1:C14, DAC1:C15, DAC1:C16, DAC1:C17: 2.7nF, SparkFun-Passives:1206
- removed DAC1:C18, DAC1:C21, PCM2707-1:C8, PCM2707-1:C9: 100uF, SparkFun-Passives:CPOL-RADIAL-100UF-25V
- removed DAC1:C7, DAC1:C8: 47uF, SparkFun-Passives:CPOL-RADIAL-100UF-25V
- removed DAC1:IC1: OPA4134UA, linear:SO14
- removed DAC1:R1: 10K, SparkFun-Passives:0805
- removed DAC1:R10, DAC1:R11, DAC1:R12, DAC1:R2, DAC1:R3, DAC1:R4, DAC1:R5, DAC1:R6, DAC1:R7, DAC1:R8: 1K, SparkFun-Passives:0805
- removed DAC1:R13, DAC1:R9: 39.2, SparkFun-Passives:0805
- removed DAC1:U$1: PCM1794A, EduAreaLib:SSOP28-0.65-10.2X5.2MM
- removed DAC1:U$6: TPA6120A2, EduAreaLib:SOIC20S
- removed PCM2707-1:C10, PCM2707-1:C11: 0.022uF, SparkFun-Passives:1206
- removed PCM2707-1:C6, PCM2707-1:C7: 1uF, SparkFun-Passives:1206
- removed PCM2707-1:J1: (no value), SparkFun-Connectors:1X04_LONGPADS
- removed PCM2707-1:J2: AUDIO_JACK_TRS_0.25"_PTH_RA, SparkFun-Connectors:AUDIO_JACK_0.25"_TRS_PTH_RA
- removed PCM2707-1:R1, PCM2707-1:R6, PCM2707-1:R9: 1M, SparkFun-Passives:0805
- removed PCM2707-1:R10, PCM2707-1:R11, PCM2707-1:R12, PCM2707-1:R13: 3.3K, SparkFun-Passives:0805
- removed PCM2707-1:R14, PCM2707-1:R15: 16, SparkFun-Passives:0805
- removed PCM2707-1:R2, PCM2707-1:R3: 22, SparkFun-Passives:0805
- removed PCM2707-1:R4: 400K, SparkFun-Passives:0805
- removed PCM2707-1:R5, PCM2707-1:R7, PCM2707-1:R8: 1.5K, SparkFun-Passives:0805
- removed PCM2707-1:U$1: PCM2707, EduAreaLib:TQFP32-0.8-7X7MM
- removed PCM2707-1:U$2: IRLML2246TRPBF, EduAreaLib:SOT23-3
- removed PCM2707-1:Y1: 12MHz CSTCE12MOG52-R0, SparkFun-Clocks:RESONATOR-SMD-3.2X1.3
- added C1, C10, C12, C19, C2, C20, C6, C9: 10uF, SparkFun-Passives:CPOL-RADIAL-100UF-25V
- added C11, C13, C22, C23, C3, C4, C5: 0.1uF, SparkFun-Passives:1206
- added C14, C15, C16, C17: 2.7nF, SparkFun-Passives:1206
- added C18, C21: 100uF, SparkFun-Passives:CPOL-RADIAL-100UF-25V
- added C7, C8: 47uF, SparkFun-Passives:CPOL-RADIAL-100UF-25V
- added IC1: OPA4134UA, linear:SO14
- added R1: 10K, SparkFun-Passives:0805
- added R10, R11, R12, R2, R3, R4, R5, R6, R7, R8: 1K, SparkFun-Passives:0805
- added R13, R9: 39.2, SparkFun-Passives:0805
- added U$1: PCM1794A, EduAreaLib:SSOP28-0.65-10.2X5.2MM
- added U$6: TPA6120A2, EduAreaLib:SOIC20S
Connections:
- removed net DAC1:!RST!: DAC1:U$1.14
- removed net DAC1:+12V: DAC1:C10.1, DAC1:C11.2, DAC1:C18.1, DAC1:C19.1, DAC1:C22.1, DAC1:IC1.4, DAC1:U$6.18, DAC1:U$6.3
- removed net DAC1:-12V: DAC1:C12.2, DAC1:C13.2, DAC1:C20.2, DAC1:C21.2, DAC1:C23.1, DAC1:IC1.11, DAC1:U$6.1, DAC1:U$6.20
- removed net DAC1:3.3V: DAC1:C10.2, DAC1:C11.1, DAC1:C12.1, DAC1:C13.1, DAC1:C2.1, DAC1:C4.2, DAC1:IC1.10, DAC1:IC1.12, DAC1:IC1.3, DAC1:IC1.5, DAC1:R10.1, DAC1:R7.1, DAC1:U$1.9
- removed net DAC1:5V: DAC1:C1.1, DAC1:C3.1, DAC1:C5.2, DAC1:C6.1, DAC1:C7.1, DAC1:C8.1, DAC1:C9.1, DAC1:U$1.15, DAC1:U$1.23, DAC1:U$1.28
- removed net DAC1:AGND: DAC1:C1.2, DAC1:C18.2, DAC1:C19.2, DAC1:C20.1, DAC1:C21.1, DAC1:C22.2, DAC1:C23.2, DAC1:C3.2, DAC1:C5.1, DAC1:C6.2, DAC1:C9.2, DAC1:R1.2, DAC1:U$1.16, DAC1:U$1.19, DAC1:U$1.24, DAC1:U$1.27
- removed net DAC1:BCK: DAC1:U$1.6
- removed net DAC1:CHSL: DAC1:U$1.2
- removed net DAC1:DATA: DAC1:U$1.5
- removed net DAC1:DEM: DAC1:U$1.3
- removed net DAC1:DGND: DAC1:C2.2, DAC1:C4.1, DAC1:U$1.8
- removed net DAC1:FMT0: DAC1:U$1.11
- removed net DAC1:FMT1: DAC1:U$1.12
- removed net DAC1:LOUT: DAC1:R9.2
- removed net DAC1:LRCK: DAC1:U$1.4
- removed net DAC1:MONO: DAC1:U$1.1
- removed net DAC1:MUTE: DAC1:U$1.10
- removed net DAC1:N$1: DAC1:C14.2, DAC1:IC1.2, DAC1:R2.1, DAC1:U$1.26
- removed net DAC1:N$10: DAC1:R10.2, DAC1:R11.2, DAC1:U$6.17
- removed net DAC1:N$11: DAC1:R12.2, DAC1:R13.1, DAC1:U$6.19
- removed net DAC1:N$14: DAC1:C15.1, DAC1:IC1.7, DAC1:R3.2, DAC1:R6.1
- removed net DAC1:N$17: DAC1:C16.2, DAC1:IC1.9, DAC1:R4.1, DAC1:U$1.18
- removed net DAC1:N$2: DAC1:C15.2, DAC1:IC1.6, DAC1:R3.1, DAC1:U$1.25
- removed net DAC1:N$20: DAC1:C16.1, DAC1:IC1.8, DAC1:R12.1, DAC1:R4.2, DAC1:U$6.16
- removed net DAC1:N$23: DAC1:C17.2, DAC1:IC1.13, DAC1:R5.1, DAC1:U$1.17
- removed net DAC1:N$25: DAC1:C17.1, DAC1:IC1.14, DAC1:R11.1, DAC1:R5.2
- removed net DAC1:N$3: DAC1:R1.1, DAC1:U$1.20
- removed net DAC1:N$4: DAC1:R6.2, DAC1:R7.2, DAC1:U$6.4
- removed net DAC1:N$5: DAC1:C7.2, DAC1:U$1.22
- removed net DAC1:N$6: DAC1:C8.2, DAC1:U$1.21
- removed net DAC1:N$8: DAC1:C14.1, DAC1:IC1.1, DAC1:R2.2, DAC1:R8.1, DAC1:U$6.5
- removed net DAC1:N$9: DAC1:R8.2, DAC1:R9.1, DAC1:U$6.2
- removed net DAC1:ROUT: DAC1:R13.2
- removed net DAC1:SYSCK: DAC1:U$1.7
- removed net DAC1:ZERO: DAC1:U$1.13
- removed net PCM2707-1:!SUSPEND!: PCM2707-1:U$1.11
- removed net PCM2707-1:3.3V: PCM2707-1:C1.1, PCM2707-1:C2.1, PCM2707-1:C3.1, PCM2707-1:C4.1, PCM2707-1:C6.2, PCM2707-1:C7.1, PCM2707-1:R7.1, PCM2707-1:R8.2, PCM2707-1:U$1.2, PCM2707-1:U$1.21, PCM2707-1:U$1.27, PCM2707-1:U$1.30
- removed net PCM2707-1:BCK: PCM2707-1:U$1.19
- removed net PCM2707-1:DGND: PCM2707-1:C1.2, PCM2707-1:C2.2, PCM2707-1:C3.2, PCM2707-1:C4.2, PCM2707-1:C5.2, PCM2707-1:C6.1, PCM2707-1:C7.2, PCM2707-1:J1.4, PCM2707-1:R1.1, PCM2707-1:U$1.1, PCM2707-1:U$1.20, PCM2707-1:U$1.25, PCM2707-1:U$1.26, PCM2707-1:U$1.31, PCM2707-1:U$1.9, PCM2707-1:Y1.2
- removed net PCM2707-1:DIN: PCM2707-1:U$1.4
- removed net PCM2707-1:DOUT: PCM2707-1:U$1.17
- removed net PCM2707-1:GNDA: PCM2707-1:J2.SLEEVE, PCM2707-1:R10.2, PCM2707-1:R11.2, PCM2707-1:R12.2, PCM2707-1:R13.2, PCM2707-1:R14.2, PCM2707-1:R15.2, PCM2707-1:U$1.16
- removed net PCM2707-1:LRCK: PCM2707-1:U$1.5
- removed net PCM2707-1:N$1: PCM2707-1:R6.1, PCM2707-1:U$1.12, PCM2707-1:Y1.1
- removed net PCM2707-1:N$10: PCM2707-1:C8.2, PCM2707-1:J2.TIP, PCM2707-1:R10.1
- removed net PCM2707-1:N$11: PCM2707-1:C9.2, PCM2707-1:J2.RING, PCM2707-1:R11.1
- removed net PCM2707-1:N$14: PCM2707-1:C10.1, PCM2707-1:R14.1
- removed net PCM2707-1:N$15: PCM2707-1:C11.1, PCM2707-1:R15.1
- removed net PCM2707-1:N$2: PCM2707-1:R5.1, PCM2707-1:U$2.3
- removed net PCM2707-1:N$3: PCM2707-1:R6.2, PCM2707-1:U$1.13, PCM2707-1:Y1.3
- removed net PCM2707-1:N$4: PCM2707-1:R2.1, PCM2707-1:U$1.23
- removed net PCM2707-1:N$5: PCM2707-1:R3.1, PCM2707-1:U$1.22
- removed net PCM2707-1:N$6: PCM2707-1:C5.1, PCM2707-1:U$1.32
- removed net PCM2707-1:N$7: PCM2707-1:R7.2, PCM2707-1:U$1.15
- removed net PCM2707-1:N$8: PCM2707-1:R8.1, PCM2707-1:U$1.10
- removed net PCM2707-1:N$9: PCM2707-1:R9.2, PCM2707-1:U$1.3
- removed net PCM2707-1:PULLUP_HANDLE: PCM2707-1:R4.2, PCM2707-1:U$2.1
- removed net PCM2707-1:SPI_!SS!: PCM2707-1:U$1.6
- removed net PCM2707-1:SPI_CLCK: PCM2707-1:U$1.7
- removed net PCM2707-1:SPI_MOSI: PCM2707-1:U$1.8
- removed net PCM2707-1:SYSCK: PCM2707-1:U$1.18
- removed net PCM2707-1:USB_D+: PCM2707-1:J1.2, PCM2707-1:R2.2, PCM2707-1:R5.2
- removed net PCM2707-1:USB_D-: PCM2707-1:J1.3, PCM2707-1:R3.2
- removed net PCM2707-1:USB_VBUS: PCM2707-1:J1.1, PCM2707-1:R1.2, PCM2707-1:R4.1, PCM2707-1:R9.1, PCM2707-1:U$1.24, PCM2707-1:U$2.2
- removed net PCM2707-1:VOUT_L: PCM2707-1:C11.2, PCM2707-1:C8.1, PCM2707-1:R13.1, PCM2707-1:U$1.28
- removed net PCM2707-1:VOUT_R: PCM2707-1:C10.2, PCM2707-1:C9.1, PCM2707-1:R12.1, PCM2707-1:U$1.29
- new net !RST!: U$1.14
- new net +12V: C10.1, C11.2, C18.1, C19.1, C22.1, IC1.4, U$6.18, U$6.3
- new net -12V: C12.2, C13.2, C20.2, C21.2, C23.1, IC1.11, U$6.1, U$6.20
- new net 3.3V: C10.2, C11.1, C12.1, C13.1, C2.1, C4.2, IC1.10, IC1.12, IC1.3, IC1.5, R10.1, R7.1, U$1.9
- new net 5V: C1.1, C3.1, C5.2, C6.1, C7.1, C8.1, C9.1, U$1.15, U$1.23, U$1.28
- new net AGND: C1.2, C18.2, C19.2, C20.1, C21.1, C22.2, C23.2, C3.2, C5.1, C6.2, C9.2, R1.2, U$1.16, U$1.19, U$1.24, U$1.27
- new net BCK: U$1.6
- new net CHSL: U$1.2
- new net DATA: U$1.5
- new net DEM: U$1.3
- new net DGND: C2.2, C4.1, U$1.8
- new net FMT0: U$1.11
- new net FMT1: U$1.12
- new net LOUT: R9.2
- new net LRCK: U$1.4
- new net MONO: U$1.1
- new net MUTE: U$1.10
- new net N$1: C14.2, IC1.2, R2.1, U$1.26
- new net N$10: R10.2, R11.2, U$6.17
- new net N$11: R12.2, R13.1, U$6.19
- new net N$14: C15.1, IC1.7, R3.2, R6.1
- new net N$17: C16.2, IC1.9, R4.1, U$1.18
- new net N$2: C15.2, IC1.6, R3.1, U$1.25
- new net N$20: C16.1, IC1.8, R12.1, R4.2, U$6.16
- new net N$23: C17.2, IC1.13, R5.1, U$1.17
- new net N$25: C17.1, IC1.14, R11.1, R5.2
- new net N$3: R1.1, U$1.20
- new net N$4: R6.2, R7.2, U$6.4
- new net N$5: C7.2, U$1.22
- new net N$6: C8.2, U$1.21
- new net N$8: C14.1, IC1.1, R2.2, R8.1, U$6.5
- new net N$9: R8.2, R9.1, U$6.2
- new net ROUT: R13.2
- new net SYSCK: U$1.7
- new net ZERO: U$1.13

Commit message: minor changes
Connections:
- new net -5V: C12.2, C13.2, IC1.11
- net +12V: no longer C10.1, C11.2, IC1.4
- net -12V: no longer C12.2, C13.2, IC1.11
- net 5V: now also C10.1, C11.2, IC1.4
Changed lines of the file:
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@@
 <drawing>
 <settings>
-<setting alwaysvectorfont="yes"/>
+<setting alwaysvectorfont="no"/>
 <setting keepoldvectorfont="yes"/>
 <setting verticaltext="up"/>
@@
 <contactref element="C8" pad="1"/>
 <contactref element="C9" pad="1"/>
-<wire x1="48.895" y1="-24.765" x2="48.895" y2="-8.255" width="0" layer="19" extent="1-1"/>
-<wire x1="29.845" y1="-24.765" x2="48.895" y2="-24.765" width="0" layer="19" extent="1-1"/>
-<wire x1="10.795" y1="-24.765" x2="29.845" y2="-24.765" width="0" layer="19" extent="1-1"/>
+<contactref element="C10" pad="1"/>
+<contactref element="C11" pad="2"/>
+<contactref element="IC1" pad="4"/>
+<wire x1="36.923" y1="-68.13" x2="27.813" y2="-77.784" width="0" layer="19" extent="1-1"/>
+<wire x1="40.173" y1="-68.13" x2="36.923" y2="-68.13" width="0" layer="19" extent="1-1"/>
+<wire x1="45.373" y1="-68.13" x2="40.173" y2="-68.13" width="0" layer="19" extent="1-1"/>
+<wire x1="49.146" y1="-69.088" x2="45.373" y2="-68.13" width="0" layer="19" extent="1-1"/>
+<wire x1="62.106" y1="-69.088" x2="49.146" y2="-69.088" width="0" layer="19" extent="1-1"/>
+<wire x1="67.186" y1="-69.088" x2="62.106" y2="-69.088" width="0" layer="19" extent="1-1"/>
+<wire x1="10.795" y1="-41.275" x2="36.923" y2="-68.13" width="0" layer="19" extent="1-1"/>
+<wire x1="10.795" y1="-24.765" x2="10.795" y2="-41.275" width="0" layer="19" extent="1-1"/>
 <wire x1="10.795" y1="-8.255" x2="10.795" y2="-24.765" width="0" layer="19" extent="1-1"/>
-<wire x1="45.373" y1="-68.13" x2="48.895" y2="-24.765" width="0" layer="19" extent="1-1"/>
-<wire x1="49.146" y1="-69.088" x2="45.373" y2="-68.13" width="0" layer="19" extent="1-1"/>
-<wire x1="40.173" y1="-68.13" x2="45.373" y2="-68.13" width="0" layer="19" extent="1-1"/>
-<wire x1="36.923" y1="-68.13" x2="40.173" y2="-68.13" width="0" layer="19" extent="1-1"/>
-<wire x1="62.106" y1="-69.088" x2="49.146" y2="-69.088" width="0" layer="19" extent="1-1"/>
+<wire x1="29.845" y1="-24.765" x2="10.795" y2="-24.765" width="0" layer="19" extent="1-1"/>
+<wire x1="48.895" y1="-24.765" x2="29.845" y2="-24.765" width="0" layer="19" extent="1-1"/>
+<wire x1="48.895" y1="-8.255" x2="48.895" y2="-24.765" width="0" layer="19" extent="1-1"/>
 </signal>
 <signal name="AGND">
@@
 <contactref element="U$6" pad="3"/>
 <contactref element="U$6" pad="18"/>
-<contactref element="C10" pad="1"/>
-<contactref element="C11" pad="2"/>
-<contactref element="IC1" pad="4"/>
 <wire x1="7.62" y1="-68.66" x2="7.62" y2="-78.66" width="0" layer="19" extent="1-1"/>
 <wire x1="10.795" y1="-57.785" x2="7.62" y2="-68.66" width="0" layer="19" extent="1-1"/>
-<wire x1="10.795" y1="-41.275" x2="10.795" y2="-57.785" width="0" layer="19" extent="1-1"/>
 <wire x1="26.54" y1="-84.201" x2="7.62" y2="-78.66" width="0" layer="19" extent="1-1"/>
-<wire x1="27.813" y1="-77.784" x2="26.54" y2="-84.201" width="0" layer="19" extent="1-1"/>
-<wire x1="48.895" y1="-41.275" x2="10.795" y2="-41.275" width="0" layer="19" extent="1-1"/>
-<wire x1="67.186" y1="-69.088" x2="48.895" y2="-41.275" width="0" layer="19" extent="1-1"/>
+<wire x1="48.895" y1="-41.275" x2="10.795" y2="-57.785" width="0" layer="19" extent="1-1"/>
 </signal>
 <signal name="-12V">
@@
 <contactref element="U$6" pad="1"/>
 <contactref element="U$6" pad="20"/>
+<wire x1="5.08" y1="-68.66" x2="5.08" y2="-78.66" width="0" layer="19" extent="1-1"/>
+<wire x1="27.305" y1="-57.785" x2="5.08" y2="-68.66" width="0" layer="19" extent="1-1"/>
+<wire x1="46.355" y1="-57.785" x2="27.305" y2="-57.785" width="0" layer="19" extent="1-1"/>
+<wire x1="31.62" y1="-84.201" x2="27.305" y2="-57.785" width="0" layer="19" extent="1-1"/>
+</signal>
+<signal name="-5V">
 <contactref element="IC1" pad="11"/>
 <contactref element="C13" pad="2"/>
 <contactref element="C12" pad="2"/>
-<wire x1="5.08" y1="-78.66" x2="3.94" y2="-84.201" width="0" layer="19" extent="1-1"/>
-<wire x1="5.08" y1="-68.66" x2="5.08" y2="-78.66" width="0" layer="19" extent="1-1"/>
-<wire x1="27.813" y1="-72.584" x2="5.08" y2="-68.66" width="0" layer="19" extent="1-1"/>
-<wire x1="31.62" y1="-84.201" x2="27.813" y2="-72.584" width="0" layer="19" extent="1-1"/>
-<wire x1="27.305" y1="-57.785" x2="27.813" y2="-72.584" width="0" layer="19" extent="1-1"/>
-<wire x1="27.305" y1="-41.275" x2="27.305" y2="-57.785" width="0" layer="19" extent="1-1"/>
-<wire x1="46.355" y1="-57.785" x2="27.305" y2="-57.785" width="0" layer="19" extent="1-1"/>
+<wire x1="27.813" y1="-72.584" x2="3.94" y2="-84.201" width="0" layer="19" extent="1-1"/>
+<wire x1="27.305" y1="-41.275" x2="27.813" y2="-72.584" width="0" layer="19" extent="1-1"/>
 </signal>
 </signals>

Commit message: minor changes
Parts:
- moved U$6 96.9 mm to (40.5, 18.5), turned to 180 degrees
- moved U$1 95.7 mm to (9.14, 18.4), turned to 270 degrees
- moved IC1 93.9 mm to (25.0, 18.7), turned to 180 degrees

Commit message: some impr
Parts:
- added J1: (no value), SparkFun-Connectors:JST-5-PTH-VERT
- added J2, J3: (no value), SparkFun-Connectors:MOLEX-1X3
- added J4: (no value), SparkFun-Connectors:MOLEX-1X2_LOCK
- added R14, R16, R18, R20: (no value), SparkFun-Passives:0805
- moved U$1 8.94 mm to (17.3, 14.8)
- moved IC1 4.59 mm to (28.1, 15.2)
Connections:
- new net GNDA: J1.1
- new net N$13: J1.4, R16.1
- new net N$16: J1.3, R18.1
- new net N$19: J1.2, R20.1
- new net N$7: J1.5, R14.1
- net !RST!: now also J4.1
- net BCK: now also R18.2
- net CHSL: now also J2.2
- net DATA: now also R16.2
- net DEM: now also J2.1
- net FMT0: now also J3.2
- net FMT1: now also J3.1
- net LRCK: now also R14.2
- net MONO: now also J2.3
- net MUTE: now also J3.3
- net SYSCK: now also R20.2
- net ZERO: now also J4.2
Routing:
- net DEM: track 0.00 -> 9.66 mm
- net CHSL: track 0.00 -> 7.72 mm
- net MONO: track 0.00 -> 6.36 mm
- net LRCK: track 0.00 -> 4.75 mm
- net SYSCK: track 0.00 -> 4.57 mm
- net DATA: track 0.00 -> 4.44 mm
- net BCK: track 0.00 -> 4.29 mm
- net N$19: track 0.00 -> 3.61 mm
- net N$16: track 0.00 -> 3.35 mm
- net N$7: track 0.00 -> 3.33 mm
- net N$13: track 0.00 -> 3.10 mm

Commit message: switched to 4 layer pcb
Parts:
- removed C10: 10uF, SparkFun-Passives:CPOL-RADIAL-100UF-25V
- removed C7: 47uF, SparkFun-Passives:CPOL-RADIAL-100UF-25V
- added J5: (no value), SparkFun-Connectors:MOLEX-1X2
- added J6, J7: (no value), SparkFun-Connectors:1X03_LONGPADS
- added J8: AUDIO_JACK_TRS_0.25"_PTH_RA, SparkFun-Connectors:AUDIO_JACK_0.25"_TRS_PTH_RA
- J1: device SparkFun-Connectors:JST-5-PTH-VERT -> SparkFun-Connectors:1X05
- moved J4 144.4 mm to (19.5, 5.50)
- moved R12 143.5 mm to (26.1, 52.1), turned to 180 degrees
- moved R13 140.5 mm to (25.3, 49.7), turned to 270 degrees
- moved C22 139.4 mm to (32.1, 55.1)
- moved R11 133.3 mm to (43.3, 47.9), turned to 180 degrees
- moved R9 131.3 mm to (22.3, 42.2), turned to 90 degrees
- moved R10 131.0 mm to (43.4, 46.1), turned to 180 degrees
- moved R7 127.9 mm to (43.4, 44.2), turned to 180 degrees
- moved R8 127.8 mm to (23.2, 39.7), turned to 180 degrees
- moved C11 127.2 mm to (38.3, 55.1)
- moved R6 125.7 mm to (43.4, 42.2), turned to 180 degrees
- moved C23 123.2 mm to (29.7, 39.0)
- moved C13 117.3 mm to (33.7, 28.9), turned to 270 degrees
- moved C14 112.6 mm to (36.8, 24.6), turned to 180 degrees
- moved R3 110.9 mm to (30.3, 27.0), turned to 180 degrees
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Connections:
- removed net AGND: C1.2, C18.2, C19.2, C20.1, C21.1, C22.2, C23.2, C3.2, C5.1, C6.2, C9.2, R1.2, U$1.16, U$1.19, U$1.24, U$1.27
- removed net GNDA: J1.1
- removed net N$20: C16.1, IC1.8, R12.1, R4.2, U$6.16
- removed net N$23: C17.2, IC1.13, R5.1, U$1.17
- new net N$12: C16.1, IC1.8, R11.1, R4.2
- net +12V: now also J7.3
- net -12V: now also J7.1
- net -5V: now also J6.1
- net 3.3V: now also J5.1; no longer C10.2, C11.1, C12.1, C13.1
- net 5V: now also J6.3; no longer C10.1, C7.1
- net DGND: now also C1.2, C11.1, C12.1, C13.1, C18.2, C19.2, C20.1, C21.1, C22.2, C23.2, C3.2, C5.1, C6.2, C9.2, J1.1, J5.2, J6.2, J7.2, J8.SLEEVE, R1.2, U$1.16, U$1.19, U$1.24, U$1.27
- net LOUT: now also J8.TIP
- net N$1: now also C15.2, IC1.6, R3.1; no longer C14.2, IC1.2, R2.1
- net N$14: now also C16.2, IC1.9, R4.1, U$1.17; no longer C15.1, IC1.7, R3.2, R6.1
- net N$17: now also C17.2, IC1.13, R5.1; no longer C16.2, IC1.9, R4.1
- net N$2: now also C14.2, IC1.2, R2.1; no longer C15.2, IC1.6, R3.1
- net N$25: now also R12.1, U$6.16; no longer R11.1
- net N$5: now also C14.1, IC1.1, R2.2, R6.1; no longer C7.2, U$1.22
- net N$6: now also U$1.22
- net N$8: now also C15.1, IC1.7, R3.2; no longer C14.1, IC1.1, R2.2
- net ROUT: now also J8.RING
Routing:
- net DGND: track 0.00 -> 120.6 mm
- net 3.3V: track 0.00 -> 70.8 mm, vias 0 -> 2
- net 5V: track 0.00 -> 54.8 mm, vias 0 -> 1
- net +12V: track 0.00 -> 45.9 mm, vias 0 -> 1
- net -5V: track 0.00 -> 39.7 mm, vias 0 -> 1
- net N$8: track 0.00 -> 36.7 mm, vias 0 -> 2
- net -12V: track 0.00 -> 24.6 mm
- net N$17: track 0.00 -> 24.2 mm
- net N$2: track 0.00 -> 24.0 mm
- net N$14: track 0.00 -> 18.5 mm
- net N$1: track 0.00 -> 18.2 mm
- net ROUT: track 0.00 -> 17.6 mm
- net ZERO: track 0.00 -> 13.1 mm
- net FMT1: track 0.00 -> 12.2 mm
- net MUTE: track 0.00 -> 11.6 mm
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Other:
- board size 160 x 100 mm -> 50 x 61 mm
