File: eagle/dac_.brd (EAGLE design)
At the start: 160 x 100 mm, 48 parts, among them IC1 OPA4134UA

Commit message: switched to 4 layer pcb
Parts:
- removed C10: 10uF, SparkFun-Passives:CPOL-RADIAL-100UF-25V
- added J7: (no value), SparkFun-Connectors:1X03_LONGPADS
- added J8: AUDIO_JACK_TRS_0.25"_PTH_RA, SparkFun-Connectors:AUDIO_JACK_0.25"_TRS_PTH_RA
- moved C22 80.9 mm to (31.4, 55.7)
- moved J6 68.7 mm to (27.9, 28.3), turned to 180 degrees
- moved C23 65.3 mm to (28.0, 39.3)
- moved C19 60.1 mm to (38.2, 37.1), turned to 270 degrees
- moved C13 59.9 mm to (33.7, 28.9), turned to 270 degrees
- moved C21 59.3 mm to (16.3, 35.2), turned to 270 degrees
- moved R13 57.9 mm to (22.9, 54.2), turned to 270 degrees
- moved R12 55.1 mm to (25.3, 54.9), turned to 180 degrees
- moved C11 50.9 mm to (36.6, 55.7), turned to 0 degrees
- moved C20 50.8 mm to (23.6, 35.1), turned to 270 degrees
- moved R9 44.7 mm to (22.3, 42.2), turned to 90 degrees
- moved C9 43.2 mm to (42.3, 52.6), turned to 90 degrees
- moved R8 40.5 mm to (23.2, 39.7), turned to 180 degrees
- moved C12 38.3 mm to (40.3, 30.4), turned to 90 degrees
- moved C18 37.1 mm to (31.4, 34.7), turned to 270 degrees
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Connections:
- removed net AGND: J6.1
- net +12V: now also J7.3
- net -12V: now also J7.1
- net -5V: now also J6.1; no longer J6.2
- net 3.3V: no longer C10.2, C11.1, C12.1, C13.1
- net 5V: no longer C10.1
- net DGND: now also C11.1, C12.1, C13.1, J6.2, J7.2, J8.SLEEVE
- net LOUT: now also J8.TIP
- net ROUT: now also J8.RING
Routing:
- net N$6: track 0.00 -> 22.9 mm, vias 0 -> 1
- net -12V: track 0.00 -> 21.0 mm
- net DGND: track 42.7 -> 24.8 mm
- net ROUT: track 0.00 -> 17.6 mm
- net N$9: track 0.00 -> 10.1 mm
- net N$25: track 6.27 -> 13.7 mm
- net N$11: track 0.00 -> 7.38 mm
- net LOUT: track 0.00 -> 5.87 mm
- net DEM: track 9.95 -> 11.9 mm
- net CHSL: track 7.98 -> 9.98 mm
- net MONO: track 6.20 -> 8.17 mm
- net ZERO: track 11.4 -> 13.1 mm
- net FMT0: track 10.1 -> 11.5 mm
- net FMT1: track 10.8 -> 12.2 mm
- net !RST!: track 9.38 -> 10.8 mm
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- added copper zone on layer 2, net DGND
Other:
- board size 160 x 100 mm -> 50 x 61 mm

Commit message: 4 layer PCB draft
Parts:
- moved R5 2.00 mm to (38.8, 10.6)
- moved C17 1.90 mm to (38.6, 12.9)
- moved C14 1.81 mm to (38.6, 24.8)
- moved R2 1.70 mm to (38.4, 27.0)
- moved C13 1.63 mm to (34.8, 30.1), turned to 180 degrees
- moved C16 1.43 mm to (28.8, 13.5)
- moved R4 1.28 mm to (29.1, 11.5)
- moved C15 0.40 mm to (30.0, 24.5)
Connections:
- net 3.3V: no longer IC1.10, IC1.12, IC1.3, IC1.5, R10.1, R7.1
- net DGND: now also IC1.10, IC1.12, IC1.3, IC1.5, R10.1, R7.1
Routing:
- net DGND: track 24.8 -> 166.8 mm, vias 0 -> 26
- net 5V: track 26.3 -> 119.6 mm, vias 1 -> 3
- net +12V: track 0.00 -> 79.6 mm, vias 0 -> 3
- net N$25: track 13.7 -> 78.1 mm, vias 0 -> 2
- net N$12: track 5.92 -> 60.7 mm
- net -5V: track 0.09 -> 48.5 mm, vias 0 -> 1
- net N$8: track 7.59 -> 44.2 mm, vias 0 -> 3
- net -12V: track 21.0 -> 47.3 mm, vias 0 -> 1
- net N$5: track 6.56 -> 28.2 mm
- net N$10: track 0.00 -> 13.6 mm
- net N$4: track 0.00 -> 13.3 mm
- net 3.3V: track 28.6 -> 18.1 mm
- net N$14: track 18.5 -> 17.6 mm
- added copper zone on layer 1, net DGND

Commit message: swap layers
Parts:
- J1: value (none) -> I2S
- J5: value (none) -> +3.3V
- J6: value (none) -> 5V/GND/-5V
- J7: value (none) -> 12V/GND/-12V
- renumbered U$1 to UK1, U$6 to UK2
Routing:
- added copper zone on layer 16, net DGND
Other:
- board text added: "Crimea/prototype/ver-2 sl@whiteants.net"
- board text added: "GND"
