File: eagle/dac-_.brd (EAGLE design)
At the start: 50 x 61 mm, 49 parts, among them IC1 OPA4134UA, J1 I2S, J5 +3.3V, J6 5V/GND/-5V, J7 12V/GND/-12V, J8 AUDIO_JACK_TRS_0.25"_PTH_RA

Commit message: repaint board
Parts:
- added R15, R17: 1K, SparkFun-Passives:0805
Connections:
- new net N$15: R15.2, R8.1, UK2.5
- new net N$18: R12.1, R17.2, UK2.16
- net N$25: now also R17.1; no longer R12.1, UK2.16
- net N$8: now also R15.1; no longer R8.1, UK2.5
Routing:
- net N$25: track 78.1 -> 76.8 mm
- net N$8: track 44.2 -> 43.2 mm
Other:
- board text added: "Crimea/prototype/ver-2 sl@whiteants.net"
- board text added: "GND"
