File: eagle/dac_.sch (EAGLE design)
At the start: 49 parts, among them IC1 OPA4134UA, J8 AUDIO_JACK_TRS_0.25"_PTH_RA

Commit message: swap layers
Parts:
- J1: value (none) -> I2S
- J5: value (none) -> +3.3V
- J6: value (none) -> 5V/GND/-5V
- J7: value (none) -> 12V/GND/-12V
- renumbered U$1 to UK1, U$6 to UK2
Other:
- moved on the sheet: J3

Commit message: repaint board
Parts:
- added R15, R17: 1K, SparkFun-Passives:RESISTOR0805-RES
- R14, R16, R18, R20: value (none) -> 27
Connections:
- new net N$15: R15.2, R8.1, UK2.LIN-
- new net N$18: R12.1, R17.2, UK2.RIN-
- net N$25: now also R17.1; no longer R12.1, UK2.RIN-
- net N$8: now also R15.1; no longer R8.1, UK2.LIN-
Changed lines of the file:
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@@
 <part name="GND10" library="supply1" library_urn="urn:adsk.eagle:library:371" deviceset="GNDA" device="" value="GND"/>
 <part name="J1" library="SparkFun-Connectors" deviceset="CONN_05" device="" value="I2S"/>
-<part name="R14" library="SparkFun-Passives" deviceset="RESISTOR" device="0805-RES"/>
-<part name="R16" library="SparkFun-Passives" deviceset="RESISTOR" device="0805-RES"/>
-<part name="R18" library="SparkFun-Passives" deviceset="RESISTOR" device="0805-RES"/>
-<part name="R20" library="SparkFun-Passives" deviceset="RESISTOR" device="0805-RES"/>
+<part name="R14" library="SparkFun-Passives" deviceset="RESISTOR" device="0805-RES" value="27"/>
+<part name="R16" library="SparkFun-Passives" deviceset="RESISTOR" device="0805-RES" value="27"/>
+<part name="R18" library="SparkFun-Passives" deviceset="RESISTOR" device="0805-RES" value="27"/>
+<part name="R20" library="SparkFun-Passives" deviceset="RESISTOR" device="0805-RES" value="27"/>
 <part name="J2" library="SparkFun-Connectors" deviceset="CONN_03" device="POLAR"/>
 <part name="J3" library="SparkFun-Connectors" deviceset="CONN_03" device="POLAR"/>
@@
 <part name="GND8" library="supply1" library_urn="urn:adsk.eagle:library:371" deviceset="GNDA" device="" value="GND"/>
 <part name="DGND" library="supply1" library_urn="urn:adsk.eagle:library:371" deviceset="GNDA" device="" value="GND"/>
+<part name="R15" library="SparkFun-Passives" deviceset="RESISTOR" device="0805-RES" value="1K"/>
+<part name="R17" library="SparkFun-Passives" deviceset="RESISTOR" device="0805-RES" value="1K"/>
 </parts>
 <sheets>
@@
 <instance part="GND10" gate="1" x="25.4" y="142.24"/>
 <instance part="J1" gate="G$1" x="15.24" y="154.94"/>
-<instance part="R14" gate="G$1" x="30.48" y="160.02"/>
-<instance part="R16" gate="G$1" x="30.48" y="157.48"/>
-<instance part="R18" gate="G$1" x="30.48" y="154.94"/>
-<instance part="R20" gate="G$1" x="30.48" y="152.4"/>
+<instance part="R14" gate="G$1" x="30.48" y="160.02" smashed="yes">
+<attribute name="NAME" x="23.368" y="160.2486" size="1.778" layer="95"/>
+<attribute name="VALUE" x="33.02" y="157.988" size="1.778" layer="96"/>
+</instance>
+<instance part="R16" gate="G$1" x="30.48" y="157.48" smashed="yes">
+<attribute name="NAME" x="23.368" y="157.7086" size="1.778" layer="95"/>
+<attribute name="VALUE" x="33.02" y="155.448" size="1.778" layer="96"/>
+</instance>
+<instance part="R18" gate="G$1" x="30.48" y="154.94" smashed="yes">
+<attribute name="NAME" x="23.368" y="155.1686" size="1.778" layer="95"/>
+<attribute name="VALUE" x="33.02" y="152.908" size="1.778" layer="96"/>
+</instance>
+<instance part="R20" gate="G$1" x="30.48" y="152.4" smashed="yes">
+<attribute name="NAME" x="23.368" y="152.6286" size="1.778" layer="95"/>
+<attribute name="VALUE" x="33.02" y="150.368" size="1.778" layer="96"/>
+</instance>
 <instance part="J2" gate="J$1" x="55.88" y="167.64"/>
 <instance part="J3" gate="J$1" x="55.88" y="152.4"/>
@@
 </instance>
 <instance part="P+1" gate="1" x="231.14" y="175.26" smashed="yes">
-<attribute name="VALUE" x="241.3" y="175.26" size="1.778" layer="96" rot="R180"/>
+<attribute name="VALUE" x="238.252" y="176.784" size="1.778" layer="96" rot="R180"/>
 </instance>
 <instance part="P-3" gate="1" x="231.14" y="160.02" smashed="yes">
-<attribute name="VALUE" x="233.68" y="165.1" size="1.778" layer="96" rot="R180"/>
+<attribute name="VALUE" x="237.49" y="161.036" size="1.778" layer="96" rot="R180"/>
 </instance>
 <instance part="AGND2" gate="VR1" x="238.76" y="165.1" smashed="yes">
-<attribute name="VALUE" x="236.22" y="165.1" size="1.778" layer="96" rot="R180"/>
+<attribute name="VALUE" x="248.412" y="166.878" size="1.778" layer="96" rot="R180"/>
 </instance>
 <instance part="GND1" gate="1" x="116.84" y="142.24"/>
@@
 <instance part="GND8" gate="1" x="187.96" y="83.82"/>
 <instance part="DGND" gate="1" x="187.96" y="104.14"/>
+<instance part="R15" gate="G$1" x="182.88" y="137.16" smashed="yes">
+<attribute name="NAME" x="177.038" y="137.6426" size="1.778" layer="95"/>
+<attribute name="VALUE" x="185.674" y="137.922" size="1.778" layer="96"/>
+</instance>
+<instance part="R17" gate="G$1" x="177.8" y="81.28" smashed="yes">
+<attribute name="NAME" x="171.958" y="81.7626" size="1.778" layer="95"/>
+<attribute name="VALUE" x="180.594" y="82.042" size="1.778" layer="96"/>
+</instance>
 </instances>
 <busses>
@@
 <net name="N$8" class="0">
 <segment>
-<pinref part="UK2" gate="G$1" pin="LIN-"/>
-<wire x1="203.2" y1="114.3" x2="193.04" y2="114.3" width="0.1524" layer="91"/>
-<wire x1="193.04" y1="114.3" x2="193.04" y2="137.16" width="0.1524" layer="91"/>
-<pinref part="R8" gate="G$1" pin="1"/>
-<wire x1="205.74" y1="137.16" x2="193.04" y2="137.16" width="0.1524" layer="91"/>
-<wire x1="193.04" y1="137.16" x2="154.94" y2="137.16" width="0.1524" layer="91"/>
-<junction x="193.04" y="137.16"/>
 <pinref part="R3" gate="G$1" pin="2"/>
 <wire x1="137.16" y1="96.52" x2="142.24" y2="96.52" width="0.1524" layer="91"/>
@@
 <junction x="142.24" y="106.68"/>
 <wire x1="154.94" y1="137.16" x2="154.94" y2="106.68" width="0.1524" layer="91"/>
+<pinref part="R15" gate="G$1" pin="1"/>
+<wire x1="177.8" y1="137.16" x2="154.94" y2="137.16" width="0.1524" layer="91"/>
 </segment>
 </net>
@@
 <junction x="142.24" y="58.42"/>
 <wire x1="165.1" y1="58.42" x2="165.1" y2="81.28" width="0.1524" layer="91"/>
-<wire x1="193.04" y1="81.28" x2="193.04" y2="93.98" width="0.1524" layer="91"/>
-<pinref part="UK2" gate="G$1" pin="RIN-"/>
-<wire x1="193.04" y1="93.98" x2="203.2" y2="93.98" width="0.1524" layer="91"/>
-<pinref part="R12" gate="G$1" pin="1"/>
-<wire x1="193.04" y1="81.28" x2="208.28" y2="81.28" width="0.1524" layer="91"/>
-<wire x1="165.1" y1="81.28" x2="193.04" y2="81.28" width="0.1524" layer="91"/>
-<junction x="193.04" y="81.28"/>
+<pinref part="R17" gate="G$1" pin="1"/>
+<wire x1="172.72" y1="81.28" x2="165.1" y2="81.28" width="0.1524" layer="91"/>
 </segment>
 </net>
@@
 </segment>
 </net>
+<net name="N$15" class="0">
+<segment>
+<pinref part="R8" gate="G$1" pin="1"/>
+<wire x1="205.74" y1="137.16" x2="193.04" y2="137.16" width="0.1524" layer="91"/>
+<pinref part="UK2" gate="G$1" pin="LIN-"/>
+<wire x1="203.2" y1="114.3" x2="193.04" y2="114.3" width="0.1524" layer="91"/>
+<wire x1="193.04" y1="114.3" x2="193.04" y2="137.16" width="0.1524" layer="91"/>
+<pinref part="R15" gate="G$1" pin="2"/>
+<wire x1="193.04" y1="137.16" x2="187.96" y2="137.16" width="0.1524" layer="91"/>
+<junction x="193.04" y="137.16"/>
+</segment>
+</net>
+<net name="N$18" class="0">
+<segment>
+<pinref part="R12" gate="G$1" pin="1"/>
+<pinref part="UK2" gate="G$1" pin="RIN-"/>
+<wire x1="193.04" y1="93.98" x2="203.2" y2="93.98" width="0.1524" layer="91"/>
+<wire x1="193.04" y1="81.28" x2="193.04" y2="93.98" width="0.1524" layer="91"/>
+<wire x1="193.04" y1="81.28" x2="208.28" y2="81.28" width="0.1524" layer="91"/>
+<pinref part="R17" gate="G$1" pin="2"/>
+<wire x1="193.04" y1="81.28" x2="182.88" y2="81.28" width="0.1524" layer="91"/>
+<junction x="193.04" y="81.28"/>
+</segment>
+</net>
